File: FPGA.kicad_sch (KiCad schematic)
At the start: 0 parts

Commit message: Second pass
Other:
- sheet Bank 34-35 ports: added DDR2_OSC, {DDR2}; removed none
Changed lines of the file:
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@@
   (title_block
     (title "PCIeDMA")
-    (date "2023-02-14")
+    (date "2024-01-01")
     (rev "1")
   )
@@
     (stroke (width 0) (type default))
   )
-  (bus (pts (xy 63.5 146.05) (xy 88.9 146.05))
+  (bus (pts (xy 62.23 148.59) (xy 88.9 148.59))
     (stroke (width 0) (type default))
   )
@@
     (stroke (width 0) (type default))
   )
+  (wire (pts (xy 114.3 147.32) (xy 139.7 147.32))
+    (stroke (width 0) (type default))
+  )
   (bus (pts (xy 76.2 123.19) (xy 88.9 123.19))
     (stroke (width 0) (type default))
@@
   (wire (pts (xy 63.5 73.66) (xy 88.9 73.66))
     (stroke (width 0) (type default))
+  )
+  (bus (pts (xy 114.3 144.78) (xy 139.7 144.78))
+    (stroke (width 0) (type default))
+  )
+  (hierarchical_label "DDR2_OSC" (shape input) (at 139.7 147.32 0) (fields_autoplaced)
+    (effects (font (size 1.27 1.27)) (justify left))
   )
   (hierarchical_label "{JTAG}" (shape bidirectional) (at 63.5 92.71 180) (fields_autoplaced)
@@
     (effects (font (size 1.27 1.27)) (justify right))
   )
-  (hierarchical_label "{USER_IO}" (shape bidirectional) (at 63.5 146.05 180) (fields_autoplaced)
+  (hierarchical_label "{DDR2}" (shape bidirectional) (at 139.7 144.78 0) (fields_autoplaced)
+    (effects (font (size 1.27 1.27)) (justify left))
+  )
+  (hierarchical_label "{USER_IO}" (shape bidirectional) (at 62.23 148.59 180) (fields_autoplaced)
     (effects (font (size 1.27 1.27)) (justify right))
   )
@@
       (effects (font (size 1.27 1.27)) (justify left top))
     )
-    (pin "{USER_IO}" bidirectional (at 88.9 146.05 180)
+    (pin "{USER_IO}" bidirectional (at 88.9 148.59 180)
       (effects (font (size 1.27 1.27)) (justify left))
     )
@@
       (effects (font (size 1.27 1.27)) (justify left))
     )
+    (pin "{DDR2}" bidirectional (at 114.3 144.78 0)
+      (effects (font (size 1.27 1.27)) (justify right))
+    )
+    (pin "DDR2_OSC" input (at 114.3 147.32 0)
+      (effects (font (size 1.27 1.27)) (justify right))
+    )
     (instances

Commit message: Third pass
Other:
- sheet Bank 15-16 ports: added {SERIAL}; removed none
- sheet Bank 34-35 ports: added {VERSION}; removed none
- company: (none) -> github.com/eggsampler
Changed lines of the file:
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@@
     (date "2024-01-01")
     (rev "1")
+    (company "github.com/eggsampler")
   )
   (junction (at 76.2 123.19) (diameter 0) (color 0 0 0 0)
@@
   )
   (bus (pts (xy 76.2 118.11) (xy 88.9 118.11))
+    (stroke (width 0) (type default))
+  )
+  (bus (pts (xy 62.23 146.05) (xy 88.9 146.05))
     (stroke (width 0) (type default))
   )
@@
     (stroke (width 0) (type default))
   )
+  (bus (pts (xy 63.5 76.2) (xy 88.9 76.2))
+    (stroke (width 0) (type default))
+  )
   (bus (pts (xy 76.2 44.45) (xy 88.9 44.45))
     (stroke (width 0) (type default))
@@
     (effects (font (size 1.27 1.27)) (justify left))
   )
+  (hierarchical_label "{SERIAL}" (shape bidirectional) (at 63.5 76.2 180) (fields_autoplaced)
+    (effects (font (size 1.27 1.27)) (justify right))
+  )
   (hierarchical_label "{JTAG}" (shape bidirectional) (at 63.5 92.71 180) (fields_autoplaced)
     (effects (font (size 1.27 1.27)) (justify right))
@@
   )
   (hierarchical_label "PCIE{I2C}" (shape bidirectional) (at 63.5 68.58 180) (fields_autoplaced)
+    (effects (font (size 1.27 1.27)) (justify right))
+  )
+  (hierarchical_label "{VERSION}" (shape bidirectional) (at 62.23 146.05 180) (fields_autoplaced)
     (effects (font (size 1.27 1.27)) (justify right))
   )
@@
       (effects (font (size 1.27 1.27)) (justify right))
     )
+    (pin "{VERSION}" bidirectional (at 88.9 146.05 180)
+      (effects (font (size 1.27 1.27)) (justify left))
+    )
     (instances
       (project "PCIeDMA"
@@
     )
   )
-  (sheet (at 88.9 63.5) (size 25.4 12.7) (fields_autoplaced)
+  (sheet (at 88.9 63.5) (size 25.4 15.24) (fields_autoplaced)
     (stroke (width 0.1524) (type solid))
     (fill (color 0 0 0 0.0000))
@@
       (effects (font (size 1.27 1.27)) (justify left bottom))
     )
-    (property "Sheetfile" "FPGA_Bank15-16.kicad_sch" (at 88.9 76.7846 0)
+    (property "Sheetfile" "FPGA_Bank15-16.kicad_sch" (at 88.9 79.3246 0)
       (effects (font (size 1.27 1.27)) (justify left top))
     )
@@
       (effects (font (size 1.27 1.27)) (justify left))
     )
+    (pin "{SERIAL}" bidirectional (at 88.9 76.2 180)
+      (effects (font (size 1.27 1.27)) (justify left))
+    )
