File: FPGA_Bank0.kicad_sch (KiCad schematic)
At the start: 14 parts, among them SW3 PROGRAM, SW4 INIT_B, U8 XC7A35T-FGG484

Commit message: Routing and layout, first pass
Parts:
- renumbered C58 to C57, R31 to R29, R32 to R30, R33 to R31, R34 to R32, R35 to R33, R36 to R34, R37 to R35, R38 to R36

Commit message: Second pass
Parts:
- renumbered D5 to D4, D4 to D5, SW4 to SW3, SW3 to SW4
Changed lines of the file:
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@@
   (title_block
     (title "PCIeDMA")
-    (date "2023-02-14")
+    (date "2024-01-01")
     (rev "1")
   )
@@
   (symbol (lib_id "Switch:SW_Push") (at 165.1 57.15 90) (unit 1)
     (in_bom yes) (on_board yes) (dnp no) (fields_autoplaced)
-    (property "Reference" "SW3" (at 166.37 55.8799 90)
+    (property "Reference" "SW4" (at 166.37 55.88 90)
       (effects (font (size 1.27 1.27)) (justify right))
     )
-    (property "Value" "PROGRAM" (at 166.37 58.4199 90)
+    (property "Value" "PROGRAM" (at 166.37 58.42 90)
       (effects (font (size 1.27 1.27)) (justify right))
     )
@@
       (project "PCIeDMA"
         (path "/e81b7940-99a9-4b7f-b36e-83163c2a41ea/1bd24438-f300-4e1e-b3e2-e79b521bfee6/53f7ad83-0234-4eaa-80d2-7167faf33ffd"
-          (reference "SW3") (unit 1)
+          (reference "SW4") (unit 1)
         )
       )
@@
   (symbol (lib_id "Device:LED_Small") (at 266.7 44.45 90) (unit 1)
     (in_bom yes) (on_board yes) (dnp no)
-    (property "Reference" "D5" (at 267.97 43.18 90)
+    (property "Reference" "D4" (at 267.97 43.18 90)
       (effects (font (size 1.27 1.27)) (justify right))
     )
@@
       (project "PCIeDMA"
         (path "/e81b7940-99a9-4b7f-b36e-83163c2a41ea/1bd24438-f300-4e1e-b3e2-e79b521bfee6/53f7ad83-0234-4eaa-80d2-7167faf33ffd"
-          (reference "D5") (unit 1)
+          (reference "D4") (unit 1)
         )
       )
@@
   (symbol (lib_id "Device:LED_Small") (at 215.9 44.45 90) (unit 1)
     (in_bom yes) (on_board yes) (dnp no)
-    (property "Reference" "D4" (at 217.17 43.18 90)
+    (property "Reference" "D5" (at 217.17 43.18 90)
       (effects (font (size 1.27 1.27)) (justify right))
     )
@@
       (project "PCIeDMA"
         (path "/e81b7940-99a9-4b7f-b36e-83163c2a41ea/1bd24438-f300-4e1e-b3e2-e79b521bfee6/53f7ad83-0234-4eaa-80d2-7167faf33ffd"
-          (reference "D4") (unit 1)
+          (reference "D5") (unit 1)
         )
       )
@@
   (symbol (lib_id "Switch:SW_Push") (at 254 57.15 90) (unit 1)
     (in_bom yes) (on_board yes) (dnp no) (fields_autoplaced)
-    (property "Reference" "SW4" (at 255.27 55.8799 90)
+    (property "Reference" "SW3" (at 255.27 55.88 90)
       (effects (font (size 1.27 1.27)) (justify right))
     )
-    (property "Value" "INIT_B" (at 255.27 58.4199 90)
+    (property "Value" "INIT_B" (at 255.27 58.42 90)
       (effects (font (size 1.27 1.27)) (justify right))
     )
@@
       (project "PCIeDMA"
         (path "/e81b7940-99a9-4b7f-b36e-83163c2a41ea/1bd24438-f300-4e1e-b3e2-e79b521bfee6/53f7ad83-0234-4eaa-80d2-7167faf33ffd"
-          (reference "SW4") (unit 1)
-        )
-      )
+          (reference "SW3") (unit 1)
+        )
+      )

Commit message: Third pass
Other:
- company: (none) -> github.com/eggsampler
Changed lines of the file:
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@@
     (date "2024-01-01")
     (rev "1")
+    (company "github.com/eggsampler")
   )
   (bus_alias "JTAG" (members "TDI" "TDO" "TCK" "TMS" "TRST"))
