File: FPGA_Bank13-14.kicad_sch (KiCad schematic)
At the start: 9 parts, among them U8 XC7A35T-FGG484

Commit message: Routing and layout, first pass
Parts:
- renumbered C59 to C58, C60 to C59, C61 to C60, C62 to C61, C63 to C62, C64 to C63, C65 to C64, R39 to R37
Changed lines of the file:
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@@
   (symbol (lib_id "Device:R_Small") (at 273.05 30.48 0) (unit 1)
     (in_bom yes) (on_board yes) (dnp no)
-    (property "Reference" "R39" (at 274.32 27.94 0)
+    (property "Reference" "R37" (at 274.32 27.94 0)
       (effects (font (size 1.27 1.27)) (justify left))
     )
@@
       (project "PCIeDMA"
         (path "/e81b7940-99a9-4b7f-b36e-83163c2a41ea/1bd24438-f300-4e1e-b3e2-e79b521bfee6/ef7f5c88-c40f-4f06-af4b-db31cadb3dc7"
-          (reference "R39") (unit 1)
+          (reference "R37") (unit 1)
         )
       )
@@
   (symbol (lib_id "Device:C_Small") (at 138.43 29.21 0) (unit 1)
     (in_bom yes) (on_board yes) (dnp no)
-    (property "Reference" "C59" (at 140.97 26.67 0)
+    (property "Reference" "C58" (at 140.97 26.67 0)
       (effects (font (size 1.27 1.27)) (justify left))
     )
@@
       (project "PCIeDMA"
         (path "/e81b7940-99a9-4b7f-b36e-83163c2a41ea/1bd24438-f300-4e1e-b3e2-e79b521bfee6/ef7f5c88-c40f-4f06-af4b-db31cadb3dc7"
-          (reference "C59") (unit 1)
+          (reference "C58") (unit 1)
         )
       )
@@
   (symbol (lib_id "Device:C_Small") (at 163.83 29.21 0) (unit 1)
     (in_bom yes) (on_board yes) (dnp no)
-    (property "Reference" "C61" (at 166.37 26.67 0)
+    (property "Reference" "C60" (at 166.37 26.67 0)
       (effects (font (size 1.27 1.27)) (justify left))
     )
@@
       (project "PCIeDMA"
         (path "/e81b7940-99a9-4b7f-b36e-83163c2a41ea/1bd24438-f300-4e1e-b3e2-e79b521bfee6/ef7f5c88-c40f-4f06-af4b-db31cadb3dc7"
-          (reference "C61") (unit 1)
+          (reference "C60") (unit 1)
         )
       )
@@
   (symbol (lib_id "Device:C_Small") (at 151.13 29.21 0) (unit 1)
     (in_bom yes) (on_board yes) (dnp no)
-    (property "Reference" "C60" (at 153.67 26.67 0)
+    (property "Reference" "C59" (at 153.67 26.67 0)
       (effects (font (size 1.27 1.27)) (justify left))
     )
@@
       (project "PCIeDMA"
         (path "/e81b7940-99a9-4b7f-b36e-83163c2a41ea/1bd24438-f300-4e1e-b3e2-e79b521bfee6/ef7f5c88-c40f-4f06-af4b-db31cadb3dc7"
-          (reference "C60") (unit 1)
+          (reference "C59") (unit 1)
         )
       )
@@
   (symbol (lib_id "Device:C_Small") (at 201.93 29.21 0) (unit 1)
     (in_bom yes) (on_board yes) (dnp no)
-    (property "Reference" "C64" (at 204.47 26.67 0)
+    (property "Reference" "C63" (at 204.47 26.67 0)
       (effects (font (size 1.27 1.27)) (justify left))
     )
@@
       (project "PCIeDMA"
         (path "/e81b7940-99a9-4b7f-b36e-83163c2a41ea/1bd24438-f300-4e1e-b3e2-e79b521bfee6/ef7f5c88-c40f-4f06-af4b-db31cadb3dc7"
-          (reference "C64") (unit 1)
+          (reference "C63") (unit 1)
         )
       )
@@
   (symbol (lib_id "PCIeDMA:+VCCO") (at 273.05 25.4 0) (unit 1)
     (in_bom yes) (on_board yes) (dnp no) (fields_autoplaced)
-    (property "Reference" "#PWR081" (at 273.05 29.21 0)
+    (property "Reference" "#PWR080" (at 273.05 29.21 0)
       (effects (font (size 1.27 1.27)) hide)
     )
@@
       (project "PCIeDMA"
         (path "/e81b7940-99a9-4b7f-b36e-83163c2a41ea/1bd24438-f300-4e1e-b3e2-e79b521bfee6/ef7f5c88-c40f-4f06-af4b-db31cadb3dc7"
-          (reference "#PWR081") (unit 1)
+          (reference "#PWR080") (unit 1)
         )
       )
@@
   (symbol (lib_id "Device:C_Small") (at 176.53 29.21 0) (unit 1)
     (in_bom yes) (on_board yes) (dnp no)
-    (property "Reference" "C62" (at 179.07 26.67 0)
+    (property "Reference" "C61" (at 179.07 26.67 0)
       (effects (font (size 1.27 1.27)) (justify left))
     )
@@
       (project "PCIeDMA"
         (path "/e81b7940-99a9-4b7f-b36e-83163c2a41ea/1bd24438-f300-4e1e-b3e2-e79b521bfee6/ef7f5c88-c40f-4f06-af4b-db31cadb3dc7"
-          (reference "C62") (unit 1)
+          (reference "C61") (unit 1)
         )
       )
@@
   (symbol (lib_id "Device:C_Small") (at 189.23 29.21 0) (unit 1)
     (in_bom yes) (on_board yes) (dnp no)
-    (property "Reference" "C63" (at 191.77 26.67 0)
+    (property "Reference" "C62" (at 191.77 26.67 0)
       (effects (font (size 1.27 1.27)) (justify left))
     )
@@
       (project "PCIeDMA"
         (path "/e81b7940-99a9-4b7f-b36e-83163c2a41ea/1bd24438-f300-4e1e-b3e2-e79b521bfee6/ef7f5c88-c40f-4f06-af4b-db31cadb3dc7"
-          (reference "C63") (unit 1)
+          (reference "C62") (unit 1)
         )
       )
@@
   (symbol (lib_id "PCIeDMA:+VCCO") (at 119.38 25.4 0) (unit 1)
     (in_bom yes) (on_board yes) (dnp no) (fields_autoplaced)
-    (property "Reference" "#PWR079" (at 119.38 29.21 0)
+    (property "Reference" "#PWR078" (at 119.38 29.21 0)
       (effects (font (size 1.27 1.27)) hide)
     )
@@
       (project "PCIeDMA"
         (path "/e81b7940-99a9-4b7f-b36e-83163c2a41ea/1bd24438-f300-4e1e-b3e2-e79b521bfee6/ef7f5c88-c40f-4f06-af4b-db31cadb3dc7"
-          (reference "#PWR079") (unit 1)
+          (reference "#PWR078") (unit 1)
         )
       )
@@
   (symbol (lib_id "power:GND") (at 138.43 33.02 0) (unit 1)
     (in_bom yes) (on_board yes) (dnp no) (fields_autoplaced)
-    (property "Reference" "#PWR080" (at 138.43 39.37 0)
+    (property "Reference" "#PWR079" (at 138.43 39.37 0)
       (effects (font (size 1.27 1.27)) hide)
     )
@@
       (project "PCIeDMA"
         (path "/e81b7940-99a9-4b7f-b36e-83163c2a41ea/1bd24438-f300-4e1e-b3e2-e79b521bfee6/ef7f5c88-c40f-4f06-af4b-db31cadb3dc7"
-          (reference "#PWR080") (unit 1)
+          (reference "#PWR079") (unit 1)
         )
       )
@@
   (symbol (lib_id "Device:C_Small") (at 214.63 29.21 0) (unit 1)
     (in_bom yes) (on_board yes) (dnp no)
-    (property "Reference" "C65" (at 217.17 26.67 0)
+    (property "Reference" "C64" (at 217.17 26.67 0)
       (effects (font (size 1.27 1.27)) (justify left))
     )
@@
       (project "PCIeDMA"
         (path "/e81b7940-99a9-4b7f-b36e-83163c2a41ea/1bd24438-f300-4e1e-b3e2-e79b521bfee6/ef7f5c88-c40f-4f06-af4b-db31cadb3dc7"
-          (reference "C65") (unit 1)
-        )
-      )
+          (reference "C64") (unit 1)
+        )
+      )

Commit message: Third pass
Other:
- company: (none) -> github.com/eggsampler
Changed lines of the file:
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@@
     (date "2024-01-01")
     (rev "1")
+    (company "github.com/eggsampler")
   )
   (bus_alias "FT601" (members "BE[0..3]" "DATA[0..31]" "CLK" "TXE" "RXF" "SIWU" "WR" "RD" "OE" "WAKEUP" "RST"))
