File: FPGA_Bank15-16.kicad_sch (KiCad schematic)
At the start: 8 parts, among them U8 XC7A35T-FGG484

Commit message: Routing and layout, first pass
Parts:
- renumbered C51 to C50, C52 to C51, C53 to C52, C54 to C53, C55 to C54, C56 to C55, C57 to C56
Changed lines of the file:
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@@
   (symbol (lib_id "Device:C_Small") (at 158.75 29.21 0) (unit 1)
     (in_bom yes) (on_board yes) (dnp no)
-    (property "Reference" "C52" (at 161.29 26.67 0)
+    (property "Reference" "C51" (at 161.29 26.67 0)
       (effects (font (size 1.27 1.27)) (justify left))
     )
@@
       (project "PCIeDMA"
         (path "/e81b7940-99a9-4b7f-b36e-83163c2a41ea/1bd24438-f300-4e1e-b3e2-e79b521bfee6/4c577754-7766-4e54-90eb-b4735aa7ae9d"
-          (reference "C52") (unit 1)
+          (reference "C51") (unit 1)
         )
       )
@@
   (symbol (lib_id "Device:C_Small") (at 222.25 29.21 0) (unit 1)
     (in_bom yes) (on_board yes) (dnp no)
-    (property "Reference" "C57" (at 224.79 26.67 0)
+    (property "Reference" "C56" (at 224.79 26.67 0)
       (effects (font (size 1.27 1.27)) (justify left))
     )
@@
       (project "PCIeDMA"
         (path "/e81b7940-99a9-4b7f-b36e-83163c2a41ea/1bd24438-f300-4e1e-b3e2-e79b521bfee6/4c577754-7766-4e54-90eb-b4735aa7ae9d"
-          (reference "C57") (unit 1)
+          (reference "C56") (unit 1)
         )
       )
@@
   (symbol (lib_id "Device:C_Small") (at 184.15 29.21 0) (unit 1)
     (in_bom yes) (on_board yes) (dnp no)
-    (property "Reference" "C54" (at 186.69 26.67 0)
+    (property "Reference" "C53" (at 186.69 26.67 0)
       (effects (font (size 1.27 1.27)) (justify left))
     )
@@
       (project "PCIeDMA"
         (path "/e81b7940-99a9-4b7f-b36e-83163c2a41ea/1bd24438-f300-4e1e-b3e2-e79b521bfee6/4c577754-7766-4e54-90eb-b4735aa7ae9d"
-          (reference "C54") (unit 1)
+          (reference "C53") (unit 1)
         )
       )
@@
   (symbol (lib_id "Device:C_Small") (at 146.05 29.21 0) (unit 1)
     (in_bom yes) (on_board yes) (dnp no)
-    (property "Reference" "C51" (at 148.59 26.67 0)
+    (property "Reference" "C50" (at 148.59 26.67 0)
       (effects (font (size 1.27 1.27)) (justify left))
     )
@@
       (project "PCIeDMA"
         (path "/e81b7940-99a9-4b7f-b36e-83163c2a41ea/1bd24438-f300-4e1e-b3e2-e79b521bfee6/4c577754-7766-4e54-90eb-b4735aa7ae9d"
-          (reference "C51") (unit 1)
+          (reference "C50") (unit 1)
         )
       )
@@
   (symbol (lib_id "power:GND") (at 146.05 33.02 0) (unit 1)
     (in_bom yes) (on_board yes) (dnp no) (fields_autoplaced)
-    (property "Reference" "#PWR066" (at 146.05 39.37 0)
+    (property "Reference" "#PWR065" (at 146.05 39.37 0)
       (effects (font (size 1.27 1.27)) hide)
     )
@@
       (project "PCIeDMA"
         (path "/e81b7940-99a9-4b7f-b36e-83163c2a41ea/1bd24438-f300-4e1e-b3e2-e79b521bfee6/4c577754-7766-4e54-90eb-b4735aa7ae9d"
-          (reference "#PWR066") (unit 1)
+          (reference "#PWR065") (unit 1)
         )
       )
@@
   (symbol (lib_id "Device:C_Small") (at 209.55 29.21 0) (unit 1)
     (in_bom yes) (on_board yes) (dnp no)
-    (property "Reference" "C56" (at 212.09 26.67 0)
+    (property "Reference" "C55" (at 212.09 26.67 0)
       (effects (font (size 1.27 1.27)) (justify left))
     )
@@
       (project "PCIeDMA"
         (path "/e81b7940-99a9-4b7f-b36e-83163c2a41ea/1bd24438-f300-4e1e-b3e2-e79b521bfee6/4c577754-7766-4e54-90eb-b4735aa7ae9d"
-          (reference "C56") (unit 1)
+          (reference "C55") (unit 1)
         )
       )
@@
   (symbol (lib_id "PCIeDMA:+VCCO") (at 146.05 25.4 0) (unit 1)
     (in_bom yes) (on_board yes) (dnp no) (fields_autoplaced)
-    (property "Reference" "#PWR065" (at 146.05 29.21 0)
+    (property "Reference" "#PWR064" (at 146.05 29.21 0)
       (effects (font (size 1.27 1.27)) hide)
     )
@@
       (project "PCIeDMA"
         (path "/e81b7940-99a9-4b7f-b36e-83163c2a41ea/1bd24438-f300-4e1e-b3e2-e79b521bfee6/4c577754-7766-4e54-90eb-b4735aa7ae9d"
-          (reference "#PWR065") (unit 1)
+          (reference "#PWR064") (unit 1)
         )
       )
@@
   (symbol (lib_id "Device:C_Small") (at 171.45 29.21 0) (unit 1)
     (in_bom yes) (on_board yes) (dnp no)
-    (property "Reference" "C53" (at 173.99 26.67 0)
+    (property "Reference" "C52" (at 173.99 26.67 0)
       (effects (font (size 1.27 1.27)) (justify left))
     )
@@
       (project "PCIeDMA"
         (path "/e81b7940-99a9-4b7f-b36e-83163c2a41ea/1bd24438-f300-4e1e-b3e2-e79b521bfee6/4c577754-7766-4e54-90eb-b4735aa7ae9d"
-          (reference "C53") (unit 1)
+          (reference "C52") (unit 1)
         )
       )
@@
   (symbol (lib_id "Device:C_Small") (at 196.85 29.21 0) (unit 1)
     (in_bom yes) (on_board yes) (dnp no)
-    (property "Reference" "C55" (at 199.39 26.67 0)
+    (property "Reference" "C54" (at 199.39 26.67 0)
       (effects (font (size 1.27 1.27)) (justify left))
     )
@@
       (project "PCIeDMA"
         (path "/e81b7940-99a9-4b7f-b36e-83163c2a41ea/1bd24438-f300-4e1e-b3e2-e79b521bfee6/4c577754-7766-4e54-90eb-b4735aa7ae9d"
-          (reference "C55") (unit 1)
-        )
-      )
+          (reference "C54") (unit 1)
+        )
+      )

Commit message: Second pass
Connections:
- net OSC: now also U8.C18 (IO_L13P_T2_MRCC_16); no longer U8.B17 (IO_L11P_T1_SRCC_16)
Changed lines of the file:
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@@
   (title_block
     (title "PCIeDMA")
-    (date "2023-02-14")
+    (date "2024-01-01")
     (rev "1")
   )
@@
   (no_connect (at 55.88 25.4))
   (no_connect (at 137.16 48.26))
-  (no_connect (at 137.16 106.68))
   (no_connect (at 58.42 25.4))
   (no_connect (at 35.56 144.78))
@@
   (no_connect (at 35.56 127))
   (no_connect (at 35.56 93.98))
+  (no_connect (at 137.16 106.68))
   (no_connect (at 137.16 78.74))
   (no_connect (at 35.56 101.6))
@@
   (no_connect (at 137.16 104.14))
   (no_connect (at 50.8 25.4))
+  (no_connect (at 137.16 99.06))
   (no_connect (at 35.56 53.34))
   (no_connect (at 35.56 137.16))
-  (no_connect (at 137.16 109.22))
   (no_connect (at 35.56 154.94))
   (no_connect (at 35.56 111.76))
@@
     (stroke (width 0) (type default))
   )
+  (wire (pts (xy 137.16 109.22) (xy 190.5 109.22))
+    (stroke (width 0) (type default))
+  )
   (wire (pts (xy 171.45 33.02) (xy 171.45 31.75))
     (stroke (width 0) (type default))
@@
   )
   (wire (pts (xy 124.46 25.4) (xy 127 25.4))
-    (stroke (width 0) (type default))
-  )
-  (wire (pts (xy 137.16 99.06) (xy 190.5 99.06))
     (stroke (width 0) (type default))
   )
@@
     (effects (font (size 1.27 1.27)) (justify left))
   )
-  (hierarchical_label "OSC" (shape input) (at 190.5 99.06 0) (fields_autoplaced)
+  (hierarchical_label "OSC" (shape input) (at 190.5 109.22 0) (fields_autoplaced)
     (effects (font (size 1.27 1.27)) (justify left))
   )

Commit message: Third pass
Connections:
- net TX: now reaches U8.D22 (IO_L22N_T3_16)
- net RX: now reaches U8.E22 (IO_L22P_T3_16)
- no-connect marks 100 -> 98
Other:
- company: (none) -> github.com/eggsampler
Changed lines of the file:
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@@
     (date "2024-01-01")
     (rev "1")
+    (company "github.com/eggsampler")
   )
   (junction (at 146.05 25.4) (diameter 0) (color 0 0 0 0)
@@
   (no_connect (at 35.56 48.26))
   (no_connect (at 137.16 137.16))
-  (no_connect (at 137.16 157.48))
   (no_connect (at 137.16 147.32))
   (no_connect (at 137.16 139.7))
@@
   (no_connect (at 35.56 160.02))
   (no_connect (at 137.16 93.98))
-  (no_connect (at 137.16 154.94))
   (no_connect (at 137.16 50.8))
   (no_connect (at 35.56 104.14))
@@
   (no_connect (at 137.16 111.76))
   (no_connect (at 53.34 25.4))
+  (bus_entry (at 149.86 157.48) (size 2.54 -2.54)
+    (stroke (width 0) (type default))
+  )
   (bus_entry (at 175.26 91.44) (size 2.54 -2.54)
     (stroke (width 0) (type default))
@@
     (stroke (width 0) (type default))
   )
+  (bus_entry (at 149.86 154.94) (size 2.54 -2.54)
+    (stroke (width 0) (type default))
+  )
   (bus_entry (at 151.13 86.36) (size 2.54 -2.54)
     (stroke (width 0) (type default))
@@
     (stroke (width 0) (type default))
   )
+  (bus (pts (xy 152.4 148.59) (xy 152.4 152.4))
+    (stroke (width 0) (type default))
+  )
   (bus (pts (xy 177.8 86.36) (xy 177.8 88.9))
     (stroke (width 0) (type default))
   )
+  (bus (pts (xy 152.4 152.4) (xy 152.4 154.94))
+    (stroke (width 0) (type default))
+  )
   (wire (pts (xy 196.85 33.02) (xy 196.85 31.75))
     (stroke (width 0) (type default))
@@
     (stroke (width 0) (type default))
   )
+  (wire (pts (xy 149.86 154.94) (xy 137.16 154.94))
+    (stroke (width 0) (type default))
+  )
   (bus (pts (xy 153.67 83.82) (xy 153.67 63.5))
     (stroke (width 0) (type default))
@@
   )
   (bus (pts (xy 177.8 76.2) (xy 177.8 86.36))
+    (stroke (width 0) (type default))
+  )
+  (wire (pts (xy 149.86 157.48) (xy 137.16 157.48))
     (stroke (width 0) (type default))
   )
@@
     (effects (font (size 1.27 1.27)) (justify right bottom))
   )
+  (label "RX" (at 149.86 154.94 180) (fields_autoplaced)
+    (effects (font (size 1.27 1.27)) (justify right bottom))
+  )
   (label "PCIE.SDA" (at 175.26 88.9 180) (fields_autoplaced)
     (effects (font (size 1.27 1.27)) (justify right bottom))
   )
+  (label "TX" (at 149.86 157.48 180) (fields_autoplaced)
+    (effects (font (size 1.27 1.27)) (justify right bottom))
+  )
   (label "PCIE.SCL" (at 175.26 91.44 180) (fields_autoplaced)
     (effects (font (size 1.27 1.27)) (justify right bottom))
@@
     (effects (font (size 1.27 1.27)) (justify left))
   )
+  (hierarchical_label "{SERIAL}" (shape bidirectional) (at 152.4 148.59 0) (fields_autoplaced)
+    (effects (font (size 1.27 1.27)) (justify left))
+  )
