File: FPGA_Bank34-35.kicad_sch (KiCad schematic)
At the start: 8 parts, among them U8 XC7A35T-FGG484

Commit message: Routing and layout, first pass
Parts:
- renumbered C66 to C65, C67 to C66, C68 to C67, C69 to C68, C70 to C69, C71 to C70, C72 to C71
Changed lines of the file:
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@@
   (symbol (lib_id "Device:C_Small") (at 60.96 22.86 0) (unit 1)
     (in_bom yes) (on_board yes) (dnp no)
-    (property "Reference" "C69" (at 63.5 20.32 0)
+    (property "Reference" "C68" (at 63.5 20.32 0)
       (effects (font (size 1.27 1.27)) (justify left))
     )
@@
       (project "PCIeDMA"
         (path "/e81b7940-99a9-4b7f-b36e-83163c2a41ea/1bd24438-f300-4e1e-b3e2-e79b521bfee6/3132f396-d655-456d-bbc5-9738228cfd9e"
-          (reference "C69") (unit 1)
+          (reference "C68") (unit 1)
         )
       )
@@
   (symbol (lib_id "Device:C_Small") (at 48.26 22.86 0) (unit 1)
     (in_bom yes) (on_board yes) (dnp no)
-    (property "Reference" "C68" (at 50.8 20.32 0)
+    (property "Reference" "C67" (at 50.8 20.32 0)
       (effects (font (size 1.27 1.27)) (justify left))
     )
@@
       (project "PCIeDMA"
         (path "/e81b7940-99a9-4b7f-b36e-83163c2a41ea/1bd24438-f300-4e1e-b3e2-e79b521bfee6/3132f396-d655-456d-bbc5-9738228cfd9e"
-          (reference "C68") (unit 1)
+          (reference "C67") (unit 1)
         )
       )
@@
   (symbol (lib_id "Device:C_Small") (at 73.66 22.86 0) (unit 1)
     (in_bom yes) (on_board yes) (dnp no)
-    (property "Reference" "C70" (at 76.2 20.32 0)
+    (property "Reference" "C69" (at 76.2 20.32 0)
       (effects (font (size 1.27 1.27)) (justify left))
     )
@@
       (project "PCIeDMA"
         (path "/e81b7940-99a9-4b7f-b36e-83163c2a41ea/1bd24438-f300-4e1e-b3e2-e79b521bfee6/3132f396-d655-456d-bbc5-9738228cfd9e"
-          (reference "C70") (unit 1)
+          (reference "C69") (unit 1)
         )
       )
@@
   (symbol (lib_id "power:GND") (at 22.86 26.67 0) (unit 1)
     (in_bom yes) (on_board yes) (dnp no) (fields_autoplaced)
-    (property "Reference" "#PWR083" (at 22.86 33.02 0)
+    (property "Reference" "#PWR082" (at 22.86 33.02 0)
       (effects (font (size 1.27 1.27)) hide)
     )
@@
       (project "PCIeDMA"
         (path "/e81b7940-99a9-4b7f-b36e-83163c2a41ea/1bd24438-f300-4e1e-b3e2-e79b521bfee6/3132f396-d655-456d-bbc5-9738228cfd9e"
-          (reference "#PWR083") (unit 1)
+          (reference "#PWR082") (unit 1)
         )
       )
@@
   (symbol (lib_id "Device:C_Small") (at 22.86 22.86 0) (unit 1)
     (in_bom yes) (on_board yes) (dnp no)
-    (property "Reference" "C66" (at 25.4 20.32 0)
+    (property "Reference" "C65" (at 25.4 20.32 0)
       (effects (font (size 1.27 1.27)) (justify left))
     )
@@
       (project "PCIeDMA"
         (path "/e81b7940-99a9-4b7f-b36e-83163c2a41ea/1bd24438-f300-4e1e-b3e2-e79b521bfee6/3132f396-d655-456d-bbc5-9738228cfd9e"
-          (reference "C66") (unit 1)
+          (reference "C65") (unit 1)
         )
       )
@@
   (symbol (lib_id "Device:C_Small") (at 35.56 22.86 0) (unit 1)
     (in_bom yes) (on_board yes) (dnp no)
-    (property "Reference" "C67" (at 38.1 20.32 0)
+    (property "Reference" "C66" (at 38.1 20.32 0)
       (effects (font (size 1.27 1.27)) (justify left))
     )
@@
       (project "PCIeDMA"
         (path "/e81b7940-99a9-4b7f-b36e-83163c2a41ea/1bd24438-f300-4e1e-b3e2-e79b521bfee6/3132f396-d655-456d-bbc5-9738228cfd9e"
-          (reference "C67") (unit 1)
+          (reference "C66") (unit 1)
         )
       )
@@
   (symbol (lib_id "PCIeDMA:+VCCO") (at 16.51 19.05 0) (unit 1)
     (in_bom yes) (on_board yes) (dnp no) (fields_autoplaced)
-    (property "Reference" "#PWR082" (at 16.51 22.86 0)
+    (property "Reference" "#PWR081" (at 16.51 22.86 0)
       (effects (font (size 1.27 1.27)) hide)
     )
@@
       (project "PCIeDMA"
         (path "/e81b7940-99a9-4b7f-b36e-83163c2a41ea/1bd24438-f300-4e1e-b3e2-e79b521bfee6/3132f396-d655-456d-bbc5-9738228cfd9e"
-          (reference "#PWR082") (unit 1)
+          (reference "#PWR081") (unit 1)
         )
       )
@@
   (symbol (lib_id "Device:C_Small") (at 86.36 22.86 0) (unit 1)
     (in_bom yes) (on_board yes) (dnp no)
-    (property "Reference" "C71" (at 88.9 20.32 0)
+    (property "Reference" "C70" (at 88.9 20.32 0)
       (effects (font (size 1.27 1.27)) (justify left))
     )
@@
       (project "PCIeDMA"
         (path "/e81b7940-99a9-4b7f-b36e-83163c2a41ea/1bd24438-f300-4e1e-b3e2-e79b521bfee6/3132f396-d655-456d-bbc5-9738228cfd9e"
-          (reference "C71") (unit 1)
+          (reference "C70") (unit 1)
         )
       )
@@
   (symbol (lib_id "Device:C_Small") (at 99.06 22.86 0) (unit 1)
     (in_bom yes) (on_board yes) (dnp no)
-    (property "Reference" "C72" (at 101.6 20.32 0)
+    (property "Reference" "C71" (at 101.6 20.32 0)
       (effects (font (size 1.27 1.27)) (justify left))
     )
@@
       (project "PCIeDMA"
         (path "/e81b7940-99a9-4b7f-b36e-83163c2a41ea/1bd24438-f300-4e1e-b3e2-e79b521bfee6/3132f396-d655-456d-bbc5-9738228cfd9e"
-          (reference "C72") (unit 1)
-        )
-      )
+          (reference "C71") (unit 1)
+        )
+      )

Commit message: Second pass
Parts:
- added C129: 47u, Capacitor_SMD:C_1206_3216Metric, symbol Device:C_Small
- added C130, C131: 4.7u, Capacitor_SMD:C_0603_1608Metric, symbol Device:C_Small
- added C132, C133, C134, C135: 0.47u, Capacitor_SMD:C_0402_1005Metric, symbol Device:C_Small
Connections:
- net GND: now also C129.2, C130.2, C131.2, C132.2, C133.2, C134.2, C135.2
- net +VCCAUX: now reaches U8.C1 (VCCO_35)
- net +VCCAUX: now also U8.F2 (VCCO_35), U8.H6 (VCCO_35), U8.J3 (VCCO_35), U8.M4 (VCCO_35), U8.N1 (VCCO_35), C129.1, C130.1, C131.1, C132.1, C133.1, C134.1, C135.1
- net ADDR4: now reaches U8.D2 (IO_L4N_T0_35)
- net ADDR8: now reaches U8.E1 (IO_L3P_T0_DQS_AD5P_35)
- net ADDR13: now reaches U8.E2 (IO_L4P_T0_35)
- net ADDR0: now reaches U8.F1 (IO_L5N_T0_AD13N_35)
- net ADDR12: now reaches U8.F3 (IO_L6P_T0_35)
- net ADDR6: now reaches U8.G1 (IO_L5P_T0_AD13P_35)
- net ADDR11: now reaches U8.G2 (IO_L8N_T1_AD14N_35)
- net ADDR7: now reaches U8.G3 (IO_L11N_T1_SRCC_35)
- net ADDR2: now reaches U8.H2 (IO_L8P_T1_AD14P_35)
- net ADDR5: now reaches U8.H3 (IO_L11P_T1_SRCC_35)
- net DDR2_OSC: now reaches U8.H4 (IO_L12P_T1_MRCC_35)
- net ADDR9: now reaches U8.H5 (IO_L10N_T1_AD15N_35)
- net ADDR10: now reaches U8.J1 (IO_L7N_T1_AD6N_35)
- net ADDR1: now reaches U8.J2 (IO_L9N_T1_DQS_AD7N_35)
- net ADDR3: now reaches U8.J4 (IO_L13N_T2_MRCC_35)
- net BA2: now reaches U8.K1 (IO_L7P_T1_AD6P_35)
- net BA0: now reaches U8.K2 (IO_L9P_T1_DQS_AD7P_35)
- net BA1: now reaches U8.K4 (IO_L13P_T2_MRCC_35)
- net CAS: now reaches U8.L1 (IO_L15N_T2_DQS_35)
- net WE: now reaches U8.L3 (IO_L14P_T2_SRCC_35)
- net CK_N: now reaches U8.L4 (IO_L18N_T2_35)
- net CK_P: now reaches U8.L5 (IO_L18P_T2_35)
- net RAS: now reaches U8.M1 (IO_L15P_T2_DQS_35)
- net DDR2.CS: now reaches U8.M2 (IO_L16N_T2_35)
- net CKE: now reaches U8.M3 (IO_L16P_T2_35)
- net DQ3: now reaches U8.M5 (IO_L23N_T3_35)
- net DQ4: now reaches U8.M6 (IO_L23P_T3_35)
- net DQ2: now reaches U8.N2 (IO_L22N_T3_35)
- net ODT: now reaches U8.N3 (IO_L19N_T3_VREF_35)
- net DM: now reaches U8.N4 (IO_L19P_T3_35)
- net DQ1: now reaches U8.N5 (IO_L24N_T3_35)
- net DQ5: now reaches U8.P1 (IO_L20N_T3_35)
- net DQ0: now reaches U8.P2 (IO_L22P_T3_35)
- net DQS_N: now reaches U8.P4 (IO_L21N_T3_DQS_35)
- net DQS_P: now reaches U8.P5 (IO_L21P_T3_DQS_35)
- net DQ6: now reaches U8.P6 (IO_L24P_T3_35)
- net DQ7: now reaches U8.R1 (IO_L20P_T3_35)
- no-connect marks 94 -> 42
Other:
- moved on the sheet: U8C

Commit message: Third pass
Connections:
- net BIT2: now reaches U8.W1 (IO_L5P_T0_34)
- net BIT0: now reaches U8.W2 (IO_L4P_T0_34)
- net BIT3: now reaches U8.Y1 (IO_L5N_T0_34)
- net BIT1: now reaches U8.Y2 (IO_L4N_T0_34)
- no-connect marks 42 -> 38
Other:
- company: (none) -> github.com/eggsampler
Changed lines of the file:
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@@
     (date "2024-01-01")
     (rev "1")
+    (company "github.com/eggsampler")
   )
   (bus_alias "USER_IO" (members "USER_SW2" "USER_SW1" "USER_LD2" "USER_LD1"))
+  (bus_alias "VERSION" (members "BIT0" "BIT1" "BIT2" "BIT3"))
   (junction (at 198.12 19.05) (diameter 0) (color 0 0 0 0)
   )
@@
   )
   (no_connect (at 53.34 68.58))
-  (no_connect (at 53.34 73.66))
   (no_connect (at 53.34 180.34))
   (no_connect (at 53.34 121.92))
@@
   (no_connect (at 53.34 99.06))
   (no_connect (at 53.34 91.44))
-  (no_connect (at 53.34 76.2))
   (no_connect (at 53.34 139.7))
   (no_connect (at 53.34 142.24))
   (no_connect (at 53.34 160.02))
   (no_connect (at 53.34 109.22))
-  (no_connect (at 53.34 78.74))
   (no_connect (at 154.94 142.24))
   (no_connect (at 53.34 119.38))
@@
   (no_connect (at 53.34 114.3))
   (no_connect (at 53.34 71.12))
-  (no_connect (at 53.34 81.28))
   (no_connect (at 53.34 137.16))
   (no_connect (at 53.34 63.5))
@@
     (stroke (width 0) (type default))
   )
+  (bus_entry (at 38.1 76.2) (size 2.54 2.54)
+    (stroke (width 0) (type default))
+  )
   (bus_entry (at 182.88 167.64) (size 2.54 -2.54)
     (stroke (width 0) (type default))
@@
     (stroke (width 0) (type default))
   )
+  (bus_entry (at 38.1 78.74) (size 2.54 2.54)
+    (stroke (width 0) (type default))
+  )
+  (bus_entry (at 38.1 73.66) (size 2.54 2.54)
+    (stroke (width 0) (type default))
+  )
   (bus_entry (at 182.88 73.66) (size 2.54 -2.54)
     (stroke (width 0) (type default))
@@
     (stroke (width 0) (type default))
   )
+  (bus_entry (at 38.1 71.12) (size 2.54 2.54)
+    (stroke (width 0) (type default))
+  )
   (wire (pts (xy 86.36 26.67) (xy 73.66 26.67))
     (stroke (width 0) (type default))
@@
     (stroke (width 0) (type default))
   )
+  (bus (pts (xy 38.1 76.2) (xy 38.1 78.74))
+    (stroke (width 0) (type default))
+  )
   (wire (pts (xy 48.26 19.05) (xy 60.96 19.05))
     (stroke (width 0) (type default))
@@
     (stroke (width 0) (type default))
   )
+  (bus (pts (xy 38.1 63.5) (xy 38.1 71.12))
+    (stroke (width 0) (type default))
+  )
   (bus (pts (xy 185.42 88.9) (xy 185.42 91.44))
     (stroke (width 0) (type default))
@@
     (stroke (width 0) (type default))
   )
+  (bus (pts (xy 38.1 71.12) (xy 38.1 73.66))
+    (stroke (width 0) (type default))
+  )
   (wire (pts (xy 154.94 177.8) (xy 182.88 177.8))
     (stroke (width 0) (type default))
@@
     (stroke (width 0) (type default))
   )
+  (wire (pts (xy 40.64 76.2) (xy 53.34 76.2))
+    (stroke (width 0) (type default))
+  )
   (wire (pts (xy 30.48 157.48) (xy 53.34 157.48))
     (stroke (width 0) (type default))
@@
     (stroke (width 0) (type default))
   )
+  (wire (pts (xy 40.64 73.66) (xy 53.34 73.66))
+    (stroke (width 0) (type default))
+  )
   (bus (pts (xy 185.42 71.12) (xy 185.42 73.66))
     (stroke (width 0) (type default))
@@
     (stroke (width 0) (type default))
   )
+  (wire (pts (xy 40.64 78.74) (xy 53.34 78.74))
+    (stroke (width 0) (type default))
+  )
   (wire (pts (xy 182.88 137.16) (xy 154.94 137.16))
     (stroke (width 0) (type default))
@@
     (stroke (width 0) (type default))
   )
+  (bus (pts (xy 38.1 73.66) (xy 38.1 76.2))
+    (stroke (width 0) (type default))
+  )
   (bus (pts (xy 27.94 180.34) (xy 27.94 182.88))
     (stroke (width 0) (type default))
@@
     (stroke (width 0) (type default))
   )
+  (wire (pts (xy 40.64 81.28) (xy 53.34 81.28))
+    (stroke (width 0) (type default))
+  )
   (wire (pts (xy 134.62 35.56) (xy 137.16 35.56))
     (stroke (width 0) (type default))
@@
     (effects (font (size 1.27 1.27)) (justify right bottom))
   )
+  (label "BIT1" (at 40.64 76.2 0) (fields_autoplaced)
+    (effects (font (size 1.27 1.27)) (justify left bottom))
+  )
   (label "ADDR13" (at 175.26 73.66 180) (fields_autoplaced)
     (effects (font (size 1.27 1.27)) (justify right bottom))
@@
     (effects (font (size 1.27 1.27)) (justify right bottom))
   )
+  (label "BIT2" (at 40.64 78.74 0) (fields_autoplaced)
+    (effects (font (size 1.27 1.27)) (justify left bottom))
+  )
   (label "ADDR4" (at 175.26 76.2 180) (fields_autoplaced)
     (effects (font (size 1.27 1.27)) (justify right bottom))
@@
     (effects (font (size 1.27 1.27)) (justify left bottom))
   )
+  (label "BIT0" (at 40.64 73.66 0) (fields_autoplaced)
+    (effects (font (size 1.27 1.27)) (justify left bottom))
+  )
   (label "ADDR9" (at 175.26 106.68 180) (fields_autoplaced)
     (effects (font (size 1.27 1.27)) (justify right bottom))
@@
   (label "BA0" (at 175.26 99.06 180) (fields_autoplaced)
     (effects (font (size 1.27 1.27)) (justify right bottom))
+  )
+  (label "BIT3" (at 40.64 81.28 0) (fields_autoplaced)
+    (effects (font (size 1.27 1.27)) (justify left bottom))
   )
   (label "ADDR6" (at 175.26 78.74 180) (fields_autoplaced)
@@
     (effects (font (size 1.27 1.27)) (justify right))
   )
+  (hierarchical_label "{VERSION}" (shape bidirectional) (at 38.1 63.5 180) (fields_autoplaced)
+    (effects (font (size 1.27 1.27)) (justify right))
+  )
