File: FPGA_BankVCC.kicad_sch (KiCad schematic)
At the start: 17 parts, among them U8 XC7A35T-FGG484

Commit message: Routing and layout, first pass
Parts:
- renumbered C73 to C72, C74 to C73, C75 to C74, C76 to C75, C77 to C76, C78 to C77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

Commit message: Third pass
Other:
- company: (none) -> github.com/eggsampler
Changed lines of the file:
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@@
     (date "2024-01-01")
     (rev "1")
+    (company "github.com/eggsampler")
   )
   (junction (at 31.75 86.36) (diameter 0) (color 0 0 0 0)
