File: FPGA_GTP.kicad_sch (KiCad schematic)
At the start: 8 parts, among them U8 XC7A35T-FGG484

Commit message: Routing and layout, first pass
Parts:
- renumbered C45 to C44, C46 to C45, C47 to C46, C48 to C47, C49 to C48, C50 to C49, R30 to R28
Connections:
- net RX0_N: now also U8.C11 (MGTPRXN1_216); no longer U8.A8 (MGTPRXN0_216)
- net RX0_P: now also U8.D11 (MGTPRXP1_216); no longer U8.B8 (MGTPRXP0_216)
- net RX1_N: now also U8.A10 (MGTPRXN2_216); no longer U8.C11 (MGTPRXN1_216)
- net RX1_P: now also U8.B10 (MGTPRXP2_216); no longer U8.D11 (MGTPRXP1_216)
- net RX2_N: now also U8.C9 (MGTPRXN3_216); no longer U8.A10 (MGTPRXN2_216)
- net RX2_P: now also U8.D9 (MGTPRXP3_216); no longer U8.B10 (MGTPRXP2_216)
- net RX3_N: now also U8.A8 (MGTPRXN0_216); no longer U8.C9 (MGTPRXN3_216)
- net RX3_P: now also U8.B8 (MGTPRXP0_216); no longer U8.D9 (MGTPRXP3_216)
- net TX0_N: now also U8.C7 (MGTPTXN3_216); no longer U8.A4 (MGTPTXN0_216)
- net TX0_P: now also U8.D7 (MGTPTXP3_216); no longer U8.B4 (MGTPTXP0_216)
- net TX1_N: now also U8.A6 (MGTPTXN2_216); no longer U8.C5 (MGTPTXN1_216)
- net TX1_P: now also U8.B6 (MGTPTXP2_216); no longer U8.D5 (MGTPTXP1_216)
- net TX2_N: now also U8.C5 (MGTPTXN1_216); no longer U8.A6 (MGTPTXN2_216)
- net TX2_P: now also U8.D5 (MGTPTXP1_216); no longer U8.B6 (MGTPTXP2_216)
- net TX3_N: now also U8.A4 (MGTPTXN0_216); no longer U8.C7 (MGTPTXN3_216)
- net TX3_P: now also U8.B4 (MGTPTXP0_216); no longer U8.D7 (MGTPTXP3_216)

Commit message: Third pass
Other:
- company: (none) -> github.com/eggsampler
Changed lines of the file:
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@@
     (date "2024-01-01")
     (rev "1")
+    (company "github.com/eggsampler")
   )
   (junction (at 186.69 53.34) (diameter 0) (color 0 0 0 0)
