File: FT601.kicad_sch (KiCad schematic)
At the start: 9 parts, among them U7 FT601Q, Y2 30MHz

Commit message: Routing and layout, first pass
Parts:
- renumbered C40 to C39, C41 to C40, C42 to C41, C43 to C42, C44 to C43, R24 to R22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
Connections:
- net DM renamed DN

Commit message: Third pass
Other:
- company: (none) -> github.com/eggsampler
Changed lines of the file:
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@@
     (date "2024-01-01")
     (rev "1")
+    (company "github.com/eggsampler")
   )
   (junction (at 87.63 146.05) (diameter 0) (color 0 0 0 0)
