File: Flash.kicad_sch (KiCad schematic)
At the start: 5 parts, among them U9 IS25WP256D-xL

Commit message: Routing and layout, first pass
Parts:
- renumbered C89 to C88, R40 to R38, R41 to R39, R42 to R40
Changed lines of the file:
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@@
   (symbol (lib_id "Device:R_Small") (at 107.95 69.85 0) (unit 1)
     (in_bom yes) (on_board yes) (dnp no)
-    (property "Reference" "R40" (at 109.22 67.31 0)
+    (property "Reference" "R38" (at 109.22 67.31 0)
       (effects (font (size 1.27 1.27)) (justify left))
     )
@@
       (project "PCIeDMA"
         (path "/e81b7940-99a9-4b7f-b36e-83163c2a41ea/9b75b021-6296-4193-9853-b9961650faa3"
+          (reference "R38") (unit 1)
+        )
+      )
+    )
+  )
+  (symbol (lib_id "PCIeDMA:+VCCO") (at 139.7 63.5 0) (unit 1)
+    (in_bom yes) (on_board yes) (dnp no) (fields_autoplaced)
+    (property "Reference" "#PWR095" (at 139.7 67.31 0)
+      (effects (font (size 1.27 1.27)) hide)
+    )
+    (property "Value" "+VCCO" (at 139.7 58.42 0)
+      (effects (font (size 1.27 1.27)))
+    )
+    (property "Footprint" "" (at 139.7 63.5 0)
+      (effects (font (size 1.27 1.27)) hide)
+    )
+    (property "Datasheet" "" (at 139.7 63.5 0)
+      (effects (font (size 1.27 1.27)) hide)
+    )
+    (pin "1")
+    (instances
+      (project "PCIeDMA"
+        (path "/e81b7940-99a9-4b7f-b36e-83163c2a41ea/9b75b021-6296-4193-9853-b9961650faa3"
+          (reference "#PWR095") (unit 1)
+        )
+      )
+    )
+  )
+  (symbol (lib_id "Device:R_Small") (at 120.65 69.85 0) (unit 1)
+    (in_bom yes) (on_board yes) (dnp no)
+    (property "Reference" "R39" (at 121.92 67.31 0)
+      (effects (font (size 1.27 1.27)) (justify left))
+    )
+    (property "Value" "1k" (at 121.92 68.58 0)
+      (effects (font (size 1 1)) (justify left))
+    )
+    (property "Footprint" "Resistor_SMD:R_0402_1005Metric" (at 120.65 69.85 0)
+      (effects (font (size 1.27 1.27)) hide)
+    )
+    (property "Datasheet" "~" (at 120.65 69.85 0)
+      (effects (font (size 1.27 1.27)) hide)
+    )
+    (property "Rating" "1/16W" (at 121.92 69.85 0)
+      (effects (font (size 1 1)) (justify left))
+    )
+    (property "Tolerance" "1%" (at 121.92 71.12 0)
+      (effects (font (size 1 1)) (justify left))
+    )
+    (property "Size" "0402" (at 121.92 72.39 0)
+      (effects (font (size 1 1)) (justify left))
+    )
+    (pin "1")
+    (pin "2")
+    (instances
+      (project "PCIeDMA"
+        (path "/e81b7940-99a9-4b7f-b36e-83163c2a41ea/9b75b021-6296-4193-9853-b9961650faa3"
+          (reference "R39") (unit 1)
+        )
+      )
+    )
+  )
+  (symbol (lib_id "Device:R_Small") (at 171.45 69.85 0) (unit 1)
+    (in_bom yes) (on_board yes) (dnp no)
+    (property "Reference" "R40" (at 172.72 67.31 0)
+      (effects (font (size 1.27 1.27)) (justify left))
+    )
+    (property "Value" "1k" (at 172.72 68.58 0)
+      (effects (font (size 1 1)) (justify left))
+    )
+    (property "Footprint" "Resistor_SMD:R_0402_1005Metric" (at 171.45 69.85 0)
+      (effects (font (size 1.27 1.27)) hide)
+    )
+    (property "Datasheet" "~" (at 171.45 69.85 0)
+      (effects (font (size 1.27 1.27)) hide)
+    )
+    (property "Rating" "1/16W" (at 172.72 69.85 0)
+      (effects (font (size 1 1)) (justify left))
+    )
+    (property "Tolerance" "1%" (at 172.72 71.12 0)
+      (effects (font (size 1 1)) (justify left))
+    )
+    (property "Size" "0402" (at 172.72 72.39 0)
+      (effects (font (size 1 1)) (justify left))
+    )
+    (pin "1")
+    (pin "2")
+    (instances
+      (project "PCIeDMA"
+        (path "/e81b7940-99a9-4b7f-b36e-83163c2a41ea/9b75b021-6296-4193-9853-b9961650faa3"
           (reference "R40") (unit 1)
-        )
-      )
-    )
-  )
-  (symbol (lib_id "PCIeDMA:+VCCO") (at 139.7 63.5 0) (unit 1)
-    (in_bom yes) (on_board yes) (dnp no) (fields_autoplaced)
-    (property "Reference" "#PWR096" (at 139.7 67.31 0)
-      (effects (font (size 1.27 1.27)) hide)
-    )
-    (property "Value" "+VCCO" (at 139.7 58.42 0)
-      (effects (font (size 1.27 1.27)))
-    )
-    (property "Footprint" "" (at 139.7 63.5 0)
-      (effects (font (size 1.27 1.27)) hide)
-    )
-    (property "Datasheet" "" (at 139.7 63.5 0)
-      (effects (font (size 1.27 1.27)) hide)
-    )
-    (pin "1")
-    (instances
-      (project "PCIeDMA"
-        (path "/e81b7940-99a9-4b7f-b36e-83163c2a41ea/9b75b021-6296-4193-9853-b9961650faa3"
-          (reference "#PWR096") (unit 1)
-        )
-      )
-    )
-  )
-  (symbol (lib_id "Device:R_Small") (at 120.65 69.85 0) (unit 1)
-    (in_bom yes) (on_board yes) (dnp no)
-    (property "Reference" "R41" (at 121.92 67.31 0)
-      (effects (font (size 1.27 1.27)) (justify left))
-    )
-    (property "Value" "1k" (at 121.92 68.58 0)
-      (effects (font (size 1 1)) (justify left))
-    )
-    (property "Footprint" "Resistor_SMD:R_0402_1005Metric" (at 120.65 69.85 0)
-      (effects (font (size 1.27 1.27)) hide)
-    )
-    (property "Datasheet" "~" (at 120.65 69.85 0)
-      (effects (font (size 1.27 1.27)) hide)
-    )
-    (property "Rating" "1/16W" (at 121.92 69.85 0)
-      (effects (font (size 1 1)) (justify left))
-    )
-    (property "Tolerance" "1%" (at 121.92 71.12 0)
-      (effects (font (size 1 1)) (justify left))
-    )
-    (property "Size" "0402" (at 121.92 72.39 0)
-      (effects (font (size 1 1)) (justify left))
-    )
-    (pin "1")
-    (pin "2")
-    (instances
-      (project "PCIeDMA"
-        (path "/e81b7940-99a9-4b7f-b36e-83163c2a41ea/9b75b021-6296-4193-9853-b9961650faa3"
-          (reference "R41") (unit 1)
-        )
-      )
-    )
-  )
-  (symbol (lib_id "Device:R_Small") (at 171.45 69.85 0) (unit 1)
-    (in_bom yes) (on_board yes) (dnp no)
-    (property "Reference" "R42" (at 172.72 67.31 0)
-      (effects (font (size 1.27 1.27)) (justify left))
-    )
-    (property "Value" "1k" (at 172.72 68.58 0)
-      (effects (font (size 1 1)) (justify left))
-    )
-    (property "Footprint" "Resistor_SMD:R_0402_1005Metric" (at 171.45 69.85 0)
-      (effects (font (size 1.27 1.27)) hide)
-    )
-    (property "Datasheet" "~" (at 171.45 69.85 0)
-      (effects (font (size 1.27 1.27)) hide)
-    )
-    (property "Rating" "1/16W" (at 172.72 69.85 0)
-      (effects (font (size 1 1)) (justify left))
-    )
-    (property "Tolerance" "1%" (at 172.72 71.12 0)
-      (effects (font (size 1 1)) (justify left))
-    )
-    (property "Size" "0402" (at 172.72 72.39 0)
-      (effects (font (size 1 1)) (justify left))
-    )
-    (pin "1")
-    (pin "2")
-    (instances
-      (project "PCIeDMA"
-        (path "/e81b7940-99a9-4b7f-b36e-83163c2a41ea/9b75b021-6296-4193-9853-b9961650faa3"
-          (reference "R42") (unit 1)
         )
       )
@@
   (symbol (lib_id "power:GND") (at 128.27 93.98 0) (unit 1)
     (in_bom yes) (on_board yes) (dnp no) (fields_autoplaced)
-    (property "Reference" "#PWR095" (at 128.27 100.33 0)
+    (property "Reference" "#PWR094" (at 128.27 100.33 0)
       (effects (font (size 1.27 1.27)) hide)
     )
@@
       (project "PCIeDMA"
         (path "/e81b7940-99a9-4b7f-b36e-83163c2a41ea/9b75b021-6296-4193-9853-b9961650faa3"
-          (reference "#PWR095") (unit 1)
+          (reference "#PWR094") (unit 1)
         )
       )
@@
   (symbol (lib_id "power:GND") (at 158.75 72.39 0) (unit 1)
     (in_bom yes) (on_board yes) (dnp no) (fields_autoplaced)
-    (property "Reference" "#PWR097" (at 158.75 78.74 0)
+    (property "Reference" "#PWR096" (at 158.75 78.74 0)
       (effects (font (size 1.27 1.27)) hide)
     )
@@
       (project "PCIeDMA"
         (path "/e81b7940-99a9-4b7f-b36e-83163c2a41ea/9b75b021-6296-4193-9853-b9961650faa3"
-          (reference "#PWR097") (unit 1)
+          (reference "#PWR096") (unit 1)
         )
       )
@@
   (symbol (lib_id "Device:C_Small") (at 158.75 69.85 0) (unit 1)
     (in_bom yes) (on_board yes) (dnp no)
-    (property "Reference" "C89" (at 161.29 67.31 0)
+    (property "Reference" "C88" (at 161.29 67.31 0)
       (effects (font (size 1.27 1.27)) (justify left))
     )
@@
       (project "PCIeDMA"
         (path "/e81b7940-99a9-4b7f-b36e-83163c2a41ea/9b75b021-6296-4193-9853-b9961650faa3"
-          (reference "C89") (unit 1)
-        )
-      )
+          (reference "C88") (unit 1)
+        )
+      )

Commit message: Third pass
Other:
- company: (none) -> github.com/eggsampler
Changed lines of the file:
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@@
     (date "2024-01-01")
     (rev "1")
+    (company "github.com/eggsampler")
   )
   (junction (at 120.65 63.5) (diameter 0) (color 0 0 0 0)
