File: Memory.kicad_sch (KiCad schematic)
At the start: 17 parts, among them U13 MT47H128M8SH-25E IT_M, X2 100MHz

Commit message: Third pass
Other:
- company: (none) -> github.com/eggsampler
Changed lines of the file:
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@@
     (date "2024-01-01")
     (rev "1")
+    (company "github.com/eggsampler")
   )
   (bus_alias "DDR2" (members "CAS" "RAS" "WE" "DDR2.CS" "ADDR[0..13]" "BA[0..3]" "CKE" "DM" "DQ[0..7]" "DQS_P" "DQS_N" "CK_P" "CK_N" "ODT"))
