File: Oscillator.kicad_sch (KiCad schematic)
At the start: 2 parts, among them X1 100MHz

Commit message: Routing and layout, first pass
Parts:
- renumbered C90 to C89
Changed lines of the file:
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@@
   (symbol (lib_id "power:GND") (at 139.7 101.6 0) (unit 1)
     (in_bom yes) (on_board yes) (dnp no) (fields_autoplaced)
-    (property "Reference" "#PWR099" (at 139.7 107.95 0)
+    (property "Reference" "#PWR098" (at 139.7 107.95 0)
       (effects (font (size 1.27 1.27)) hide)
     )
@@
       (project "PCIeDMA"
         (path "/e81b7940-99a9-4b7f-b36e-83163c2a41ea/fb8eb311-0296-43ff-b679-9d680dd559f1"
-          (reference "#PWR099") (unit 1)
+          (reference "#PWR098") (unit 1)
         )
       )
@@
   (symbol (lib_id "Device:C_Small") (at 120.65 83.82 0) (mirror y) (unit 1)
     (in_bom yes) (on_board yes) (dnp no)
-    (property "Reference" "C90" (at 118.11 81.28 0)
+    (property "Reference" "C89" (at 118.11 81.28 0)
       (effects (font (size 1.27 1.27)) (justify left))
     )
@@
       (project "PCIeDMA"
         (path "/e81b7940-99a9-4b7f-b36e-83163c2a41ea/fb8eb311-0296-43ff-b679-9d680dd559f1"
-          (reference "C90") (unit 1)
+          (reference "C89") (unit 1)
         )
       )
@@
   (symbol (lib_id "PCIeDMA:+VCCO") (at 139.7 76.2 0) (unit 1)
     (in_bom yes) (on_board yes) (dnp no) (fields_autoplaced)
-    (property "Reference" "#PWR098" (at 139.7 80.01 0)
+    (property "Reference" "#PWR097" (at 139.7 80.01 0)
       (effects (font (size 1.27 1.27)) hide)
     )
@@
       (project "PCIeDMA"
         (path "/e81b7940-99a9-4b7f-b36e-83163c2a41ea/fb8eb311-0296-43ff-b679-9d680dd559f1"
-          (reference "#PWR098") (unit 1)
+          (reference "#PWR097") (unit 1)
         )
       )

Commit message: Third pass
Other:
- company: (none) -> github.com/eggsampler
Changed lines of the file:
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@@
     (date "2024-01-01")
     (rev "1")
+    (company "github.com/eggsampler")
   )
   (junction (at 139.7 99.06) (diameter 0) (color 0 0 0 0)
