File: PCIe4x.kicad_sch (KiCad schematic)
At the start: 34 parts, among them J1 PCIe_x4, M1 PCIe_Bracket

Commit message: Routing and layout, first pass
Connections:
- net RX0_N: now also C1.1; no longer C4.1
- net RX0_P: now also C5.1; no longer C8.1
- net RX1_N: now also C2.1; no longer C1.1
- net RX1_P: now also C6.1; no longer C5.1
- net RX2_N: now also C3.1; no longer C2.1
- net RX2_P: now also C7.1; no longer C6.1
- net RX3_N: now also C4.1; no longer C3.1
- net RX3_P: now also C8.1; no longer C7.1
- net TX0_N: now also C15.2; no longer C18.2
- net TX0_P: now also C10.2; no longer C13.2
- net TX1_N: now also C16.2; no longer C17.2
- net TX1_P: now also C11.2; no longer C12.2
- net TX2_N: now also C17.2; no longer C16.2
- net TX2_P: now also C12.2; no longer C11.2
- net TX3_N: now also C18.2; no longer C15.2
- net TX3_P: now also C13.2; no longer C10.2
Changed lines of the file:
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@@
     (effects (font (size 1.27 1.27)) (justify right bottom))
   )
-  (label "TX0_P" (at 162.56 129.54 180) (fields_autoplaced)
+  (label "RX1_N" (at 27.94 106.68 0) (fields_autoplaced)
+    (effects (font (size 1.27 1.27)) (justify left bottom))
+  )
+  (label "TX1_N" (at 162.56 111.76 180) (fields_autoplaced)
     (effects (font (size 1.27 1.27)) (justify right bottom))
   )
@@
     (effects (font (size 1.27 1.27)) (justify left bottom))
   )
-  (label "TX1_N" (at 162.56 121.92 180) (fields_autoplaced)
-    (effects (font (size 1.27 1.27)) (justify right bottom))
-  )
   (label "PER0_P" (at 120.65 93.98 0) (fields_autoplaced)
     (effects (font (size 1.27 1.27)) (justify left bottom))
   )
   (label "PER3_N" (at 120.65 132.08 0) (fields_autoplaced)
-    (effects (font (size 1.27 1.27)) (justify left bottom))
-  )
-  (label "RX1_N" (at 27.94 91.44 0) (fields_autoplaced)
     (effects (font (size 1.27 1.27)) (justify left bottom))
   )
@@
     (effects (font (size 1.27 1.27)) (justify right bottom))
   )
-  (label "RX0_P" (at 27.94 124.46 0) (fields_autoplaced)
-    (effects (font (size 1.27 1.27)) (justify left bottom))
-  )
   (label "CLK_N" (at 162.4343 88.9 180) (fields_autoplaced)
-    (effects (font (size 1.27 1.27)) (justify right bottom))
-  )
-  (label "RX2_P" (at 27.94 104.14 0) (fields_autoplaced)
-    (effects (font (size 1.27 1.27)) (justify left bottom))
-  )
-  (label "TX1_P" (at 162.56 119.38 180) (fields_autoplaced)
     (effects (font (size 1.27 1.27)) (justify right bottom))
   )
@@
     (effects (font (size 1.27 1.27)) (justify right bottom))
   )
-  (label "TX2_N" (at 162.56 111.76 180) (fields_autoplaced)
+  (label "TX3_N" (at 162.56 132.08 180) (fields_autoplaced)
     (effects (font (size 1.27 1.27)) (justify right bottom))
   )
-  (label "TX3_N" (at 162.56 96.52 180) (fields_autoplaced)
-    (effects (font (size 1.27 1.27)) (justify right bottom))
+  (label "RX3_N" (at 27.94 127 0) (fields_autoplaced)
+    (effects (font (size 1.27 1.27)) (justify left bottom))
   )
   (label "REFCLK+" (at 120.65 86.36 0) (fields_autoplaced)
-    (effects (font (size 1.27 1.27)) (justify left bottom))
-  )
-  (label "RX0_N" (at 27.999 127 0) (fields_autoplaced)
     (effects (font (size 1.27 1.27)) (justify left bottom))
   )
@@
     (effects (font (size 1.27 1.27)) (justify left bottom))
   )
-  (label "RX1_P" (at 28.0067 88.9 0) (fields_autoplaced)
-    (effects (font (size 1.27 1.27)) (justify left bottom))
-  )
-  (label "RX3_N" (at 27.94 116.84 0) (fields_autoplaced)
-    (effects (font (size 1.27 1.27)) (justify left bottom))
-  )
   (label "SCL_SJ" (at 68.58 63.5 0) (fields_autoplaced)
     (effects (font (size 1.27 1.27)) (justify left bottom))
-  )
-  (label "TX3_P" (at 162.56 93.98 180) (fields_autoplaced)
-    (effects (font (size 1.27 1.27)) (justify right bottom))
   )
   (label "REFCLK-" (at 120.65 88.9 0) (fields_autoplaced)
     (effects (font (size 1.27 1.27)) (justify left bottom))
   )
+  (label "TX0_P" (at 162.56 93.98 180) (fields_autoplaced)
+    (effects (font (size 1.27 1.27)) (justify right bottom))
+  )
   (label "CLK_P" (at 162.56 86.36 180) (fields_autoplaced)
     (effects (font (size 1.27 1.27)) (justify right bottom))
   )
-  (label "RX3_P" (at 27.94 114.3 0) (fields_autoplaced)
+  (label "RX1_P" (at 28.0067 104.14 0) (fields_autoplaced)
     (effects (font (size 1.27 1.27)) (justify left bottom))
   )
@@
     (effects (font (size 1.27 1.27)) (justify right bottom))
   )
-  (label "TX2_P" (at 162.56 109.22 180) (fields_autoplaced)
-    (effects (font (size 1.27 1.27)) (justify right bottom))
-  )
   (label "PET2_P" (at 69.85 114.3 180) (fields_autoplaced)
     (effects (font (size 1.27 1.27)) (justify right bottom))
   )
   (label "PER0_N" (at 120.65 96.52 0) (fields_autoplaced)
+    (effects (font (size 1.27 1.27)) (justify left bottom))
+  )
+  (label "TX2_N" (at 162.56 121.92 180) (fields_autoplaced)
+    (effects (font (size 1.27 1.27)) (justify right bottom))
+  )
+  (label "TX3_P" (at 162.56 129.54 180) (fields_autoplaced)
+    (effects (font (size 1.27 1.27)) (justify right bottom))
+  )
+  (label "TX0_N" (at 162.56 96.52 180) (fields_autoplaced)
+    (effects (font (size 1.27 1.27)) (justify right bottom))
+  )
+  (label "RX2_N" (at 27.999 116.84 0) (fields_autoplaced)
     (effects (font (size 1.27 1.27)) (justify left bottom))
   )
@@
     (effects (font (size 1.27 1.27)) (justify right bottom))
   )
-  (label "TX0_N" (at 162.56 132.08 180) (fields_autoplaced)
+  (label "RX0_N" (at 27.999 91.44 0) (fields_autoplaced)
+    (effects (font (size 1.27 1.27)) (justify left bottom))
+  )
+  (label "RX2_P" (at 27.94 114.3 0) (fields_autoplaced)
+    (effects (font (size 1.27 1.27)) (justify left bottom))
+  )
+  (label "TX2_P" (at 162.56 119.38 180) (fields_autoplaced)
     (effects (font (size 1.27 1.27)) (justify right bottom))
+  )
+  (label "RX3_P" (at 27.94 124.46 0) (fields_autoplaced)
+    (effects (font (size 1.27 1.27)) (justify left bottom))
   )
   (label "PERST" (at 162.4343 78.74 180) (fields_autoplaced)
@@
     (effects (font (size 1.27 1.27)) (justify right bottom))
   )
-  (label "RX2_N" (at 27.999 106.68 0) (fields_autoplaced)
-    (effects (font (size 1.27 1.27)) (justify left bottom))
-  )
   (label "SDA_SJ" (at 68.58 66.04 0) (fields_autoplaced)
     (effects (font (size 1.27 1.27)) (justify left bottom))
@@
     (effects (font (size 1.27 1.27)) (justify right bottom))
   )
+  (label "TX1_P" (at 162.56 109.22 180) (fields_autoplaced)
+    (effects (font (size 1.27 1.27)) (justify right bottom))
+  )
+  (label "RX0_P" (at 27.94 88.9 0) (fields_autoplaced)
+    (effects (font (size 1.27 1.27)) (justify left bottom))
+  )
   (label "PER2_N" (at 120.65 121.92 0) (fields_autoplaced)

Commit message: Second pass
Connections:
- net +3.3VA is gone; now on net +3.3V: J1.B8 (+3.3V)
- net +3.3V: no longer J1.B10 (+3.3V_aux)
- no-connect marks 6 -> 7

Commit message: Third pass
Parts:
- removed JP1, JP2, JP3, JP4: SolderJumper_2_Bridged, Jumper:SolderJumper-2_P1.3mm_Bridged_RoundedPad1.0x1.5mm, symbol Jumper:SolderJumper_2_Bridged
- added SW6: A6H-4101, Button_Switch_SMD:SW_DIP_SPSTx04_Slide_Omron_A6H-4101_W6.15mm_P1.27mm, symbol Switch:SW_DIP_x04
Connections:
- net PCIE.SCL: now also SW6.1
- net PCIE.SDA: now also SW6.2
- net PERST_R: now also SW6.3
- net PERST_SJ: now also SW6.6
- net SCL_SJ: now also SW6.8
- net SDA_SJ: now also SW6.7
- net WAKE_R: now also SW6.4
- net WAKE_SJ: now also SW6.5
Other:
- company: (none) -> github.com/eggsampler

Commit message: another quick pass
Parts:
- J1: footprint PCIeDMA:BUS_PCIexpress_x4 -> Connector_PCBEdge:BUS_PCIexpress_x4
Connections:
- net PERST_SJ renamed PERST_PCIE
- net SCL_SJ renamed SCL_PCIE
- net SDA_SJ renamed SDA_PCIE
- net WAKE_SJ renamed WAKE_PCIE
Other:
- note added: "Notes: ------------ DIP Switches for enabling/disabling hardware lines"
