File: PCIeDMA.kicad_sch (KiCad schematic)
At the start: 0 parts

Commit message: Second pass
Other:
- added sheet Memory (Memory.kicad_sch)
- sheet FPGA ports: added DDR2_OSC, {DDR2}; removed none

Commit message: Third pass
Parts:
- added NT1, NT2: NetTie_2, NetTie:NetTie-2_SMD_Pad0.5mm, symbol Device:NetTie_2
Connections:
- new net +VCCO: NT1.2
- new net BIT0: NT1.1
- new net BIT1: NT2.1
- new net GND: NT2.2
Other:
- sheet FPGA ports: added {SERIAL}, {VERSION}; removed none
- sheet USB JTAG ports: added {SERIAL}; removed none
- company: (none) -> github.com/eggsampler
Changed lines of the file:
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@@
     (date "2024-01-01")
     (rev "1")
-  )
-  (bus_entry (at 73.66 76.2) (size 2.54 -2.54)
+    (company "github.com/eggsampler")
+  )
+  (junction (at 154.94 160.02) (diameter 0) (color 0 0 0 0)
+  )
+  (junction (at 154.94 162.56) (diameter 0) (color 0 0 0 0)
+  )
+  (bus_entry (at 139.7 152.4) (size 2.54 2.54)
+    (stroke (width 0) (type default))
+  )
+  (bus_entry (at 139.7 154.94) (size 2.54 2.54)
+    (stroke (width 0) (type default))
+  )
+  (bus_entry (at 139.7 157.48) (size 2.54 2.54)
+    (stroke (width 0) (type default))
+  )
+  (bus_entry (at 139.7 160.02) (size 2.54 2.54)
+    (stroke (width 0) (type default))
+  )
+  (bus_entry (at 73.66 73.66) (size 2.54 -2.54)
     (stroke (width 0) (type default))
   )
@@
     (stroke (width 0) (type default))
   )
+  (bus (pts (xy 139.7 152.4) (xy 139.7 154.94))
+    (stroke (width 0) (type default))
+  )
   (wire (pts (xy 127 76.2) (xy 177.8 76.2))
     (stroke (width 0) (type default))
@@
     (stroke (width 0) (type default))
   )
-  (bus (pts (xy 73.66 76.2) (xy 100.33 76.2))
+  (wire (pts (xy 154.94 162.56) (xy 162.56 162.56))
+    (stroke (width 0) (type default))
+  )
+  (wire (pts (xy 142.24 154.94) (xy 162.56 154.94))
+    (stroke (width 0) (type default))
+  )
+  (wire (pts (xy 167.64 162.56) (xy 177.8 162.56))
+    (stroke (width 0) (type default))
+  )
+  (bus (pts (xy 73.66 73.66) (xy 100.33 73.66))
     (stroke (width 0) (type default))
   )
@@
     (stroke (width 0) (type default))
   )
-  (wire (pts (xy 76.2 73.66) (xy 76.2 57.15))
-    (stroke (width 0) (type default))
-  )
-  (bus (pts (xy 50.8 76.2) (xy 73.66 76.2))
+  (bus (pts (xy 50.8 78.74) (xy 100.33 78.74))
+    (stroke (width 0) (type default))
+  )
+  (wire (pts (xy 76.2 71.12) (xy 76.2 57.15))
+    (stroke (width 0) (type default))
+  )
+  (wire (pts (xy 142.24 160.02) (xy 154.94 160.02))
+    (stroke (width 0) (type default))
+  )
+  (bus (pts (xy 139.7 157.48) (xy 139.7 160.02))
+    (stroke (width 0) (type default))
+  )
+  (wire (pts (xy 142.24 157.48) (xy 154.94 157.48))
+    (stroke (width 0) (type default))
+  )
+  (bus (pts (xy 50.8 73.66) (xy 73.66 73.66))
+    (stroke (width 0) (type default))
+  )
+  (wire (pts (xy 154.94 157.48) (xy 154.94 160.02))
     (stroke (width 0) (type default))
   )
@@
     (stroke (width 0) (type default))
   )
+  (bus (pts (xy 139.7 154.94) (xy 139.7 157.48))
+    (stroke (width 0) (type default))
+  )
+  (wire (pts (xy 154.94 160.02) (xy 154.94 162.56))
+    (stroke (width 0) (type default))
+  )
+  (wire (pts (xy 167.64 154.94) (xy 177.8 154.94))
+    (stroke (width 0) (type default))
+  )
+  (bus (pts (xy 127 152.4) (xy 139.7 152.4))
+    (stroke (width 0) (type default))
+  )
   (bus (pts (xy 127 113.03) (xy 177.8 113.03))
     (stroke (width 0) (type default))
@@
     (stroke (width 0) (type default))
   )
+  (wire (pts (xy 142.24 162.56) (xy 154.94 162.56))
+    (stroke (width 0) (type default))
+  )
   (bus (pts (xy 50.8 152.4) (xy 100.33 152.4))
     (stroke (width 0) (type default))
@@
   (bus (pts (xy 50.8 114.3) (xy 100.33 114.3))
     (stroke (width 0) (type default))
+  )
+  (label "BIT2" (at 142.24 160.02 0) (fields_autoplaced)
+    (effects (font (size 1.27 1.27)) (justify left bottom))
   )
   (label "TRST" (at 76.2 57.15 0) (fields_autoplaced)
     (effects (font (size 1.27 1.27)) (justify left bottom))
   )
+  (label "BIT3" (at 142.24 162.56 0) (fields_autoplaced)
+    (effects (font (size 1.27 1.27)) (justify left bottom))
+  )
+  (label "BIT1" (at 142.24 157.48 0) (fields_autoplaced)
+    (effects (font (size 1.27 1.27)) (justify left bottom))
+  )
+  (label "BIT0" (at 142.24 154.94 0) (fields_autoplaced)
+    (effects (font (size 1.27 1.27)) (justify left bottom))
+  )
+  (symbol (lib_id "Device:NetTie_2") (at 165.1 154.94 0) (unit 1)
+    (in_bom no) (on_board yes) (dnp no) (fields_autoplaced)
+    (property "Reference" "NT1" (at 165.1 149.86 0)
+      (effects (font (size 1.27 1.27)))
+    )
+    (property "Value" "NetTie_2" (at 165.1 152.4 0)
+      (effects (font (size 1.27 1.27)))
+    )
+    (property "Footprint" "NetTie:NetTie-2_SMD_Pad0.5mm" (at 165.1 154.94 0)
+      (effects (font (size 1.27 1.27)) hide)
+    )
+    (property "Datasheet" "~" (at 165.1 154.94 0)
+      (effects (font (size 1.27 1.27)) hide)
+    )
+    (pin "2")
+    (pin "1")
+    (instances
+      (project "PCIeDMA"
+        (path "/e81b7940-99a9-4b7f-b36e-83163c2a41ea"
+          (reference "NT1") (unit 1)
+        )
+      )
+    )
+  )
+  (symbol (lib_id "power:GND") (at 177.8 162.56 0) (unit 1)
+    (in_bom yes) (on_board yes) (dnp no) (fields_autoplaced)
+    (property "Reference" "#PWR0183" (at 177.8 168.91 0)
+      (effects (font (size 1.27 1.27)) hide)
+    )
+    (property "Value" "GND" (at 177.8 167.64 0)
+      (effects (font (size 1.27 1.27)))
+    )
+    (property "Footprint" "" (at 177.8 162.56 0)
+      (effects (font (size 1.27 1.27)) hide)
+    )
+    (property "Datasheet" "" (at 177.8 162.56 0)
+      (effects (font (size 1.27 1.27)) hide)
+    )
+    (pin "1")
+    (instances
+      (project "PCIeDMA"
+        (path "/e81b7940-99a9-4b7f-b36e-83163c2a41ea"
+          (reference "#PWR0183") (unit 1)
+        )
+      )
+    )
+  )
+  (symbol (lib_id "Device:NetTie_2") (at 165.1 162.56 0) (unit 1)
+    (in_bom no) (on_board yes) (dnp no) (fields_autoplaced)
+    (property "Reference" "NT2" (at 165.1 157.48 0)
+      (effects (font (size 1.27 1.27)))
+    )
+    (property "Value" "NetTie_2" (at 165.1 160.02 0)
+      (effects (font (size 1.27 1.27)))
+    )
+    (property "Footprint" "NetTie:NetTie-2_SMD_Pad0.5mm" (at 165.1 162.56 0)
+      (effects (font (size 1.27 1.27)) hide)
+    )
+    (property "Datasheet" "~" (at 165.1 162.56 0)
+      (effects (font (size 1.27 1.27)) hide)
+    )
+    (pin "2")
+    (pin "1")
+    (instances
+      (project "PCIeDMA"
+        (path "/e81b7940-99a9-4b7f-b36e-83163c2a41ea"
+          (reference "NT2") (unit 1)
+        )
+      )
+    )
+  )
+  (symbol (lib_id "PCIeDMA:+VCCO") (at 177.8 154.94 0) (unit 1)
+    (in_bom yes) (on_board yes) (dnp no) (fields_autoplaced)
+    (property "Reference" "#PWR0182" (at 177.8 158.75 0)
+      (effects (font (size 1.27 1.27)) hide)
+    )
+    (property "Value" "+VCCO" (at 177.8 149.86 0)
+      (effects (font (size 1.27 1.27)))
+    )
+    (property "Footprint" "" (at 177.8 154.94 0)
+      (effects (font (size 1.27 1.27)) hide)
+    )
+    (property "Datasheet" "" (at 177.8 154.94 0)
+      (effects (font (size 1.27 1.27)) hide)
+    )
+    (pin "1")
+    (instances
+      (project "PCIeDMA"
+        (path "/e81b7940-99a9-4b7f-b36e-83163c2a41ea"
+          (reference "#PWR0182") (unit 1)
+        )
+      )
+    )
+  )
   (sheet (at 241.3 25.4) (size 25.4 25.4) (fields_autoplaced)
     (stroke (width 0.1524) (type solid))
@@
       (effects (font (size 1.27 1.27)) (justify left))
     )
-    (pin "{JTAG}" bidirectional (at 100.33 76.2 180)
+    (pin "{JTAG}" bidirectional (at 100.33 73.66 180)
       (effects (font (size 1.27 1.27)) (justify left))
     )
@@
       (effects (font (size 1.27 1.27)) (justify right))
     )
+    (pin "{SERIAL}" bidirectional (at 100.33 78.74 180)
+      (effects (font (size 1.27 1.27)) (justify left))
+    )
+    (pin "{VERSION}" bidirectional (at 127 152.4 0)
+      (effects (font (size 1.27 1.27)) (justify right))
+    )
     (instances
       (project "PCIeDMA"
@@
       (effects (font (size 1.27 1.27)) (justify left top))
     )
-    (pin "{JTAG}" bidirectional (at 50.8 76.2 0)
-      (effects (font (size 1.27 1.27)) (justify right))
-    )
+    (pin "{JTAG}" bidirectional (at 50.8 73.66 0)
+      (effects (font (size 1.27 1.27)) (justify right))
+    )
+    (pin "{SERIAL}" bidirectional (at 50.8 78.74 0)
+      (effects (font (size 1.27 1.27)) (justify right))
+    )
