File: PowerBoard.kicad_sch (KiCad schematic)
At the start: 30 parts, among them Q2 Q_NMOS_GDS, Q3 Q_PMOS_GDS, Q4 Q_PMOS_GDS, SW5 SW_SPDT, U10 MT2492, U11 MT2492

Commit message: Routing and layout, first pass
Parts:
- renumbered C101 to C100, C91 to C90, C92 to C91, C93 to C92, C94 to C93, C95 to C94, C96 to C95, C97 to C96, C98 to C97, C99 to C98, C100 to C99, Q2 to Q1, Q3 to Q2, Q4 to Q3, R43 to R41, R44 to R42, R45 to R43, R46 to R44, R47 to R45, R48 to R46, R49 to R47, R50 to R48, R51 to R49, R52 to R50, R53 to R51

Commit message: Second pass
Parts:
- removed Q1: Q_NMOS_GDS, Package_TO_SOT_SMD:SOT-23, symbol Device:Q_NMOS_GDS
- added Q1: 2N7002, Package_TO_SOT_SMD:SOT-23, symbol Transistor_FET:2N7002
- Q2, Q3: value Q_PMOS_GDS -> AO3401A
- R50: value 100k -> 10k
Connections:
- net +12V: no longer R50.1
- net 5VJT_SW_EN: now also Q1.3 (D)
- net GND: now also Q1.2 (S)
- net at R45.2, R46.1: now also Q1.1 (G)
- net 5V_SW_EN renamed 12V_SW_EN
- net 12V_SW_EN: now also R50.1
Other:
- note added: "JTAG 3v3 Power Enable"
- note added: "JTAG 3v3 Power Supply"
- note added: "JTAG 5v Power Select"
- note added: "Main Power Switch"
- note added: "Notes: ------------ This should allow the board 5v to be powered from the jtag supply if the 12v isn't present ie card not plugged in, or the switch is off, and provide some reverse polarity protection. TODO: Size some mosfets, maybe dual package so8?"
- note added: "Notes: ------------ This will enable the 3v3 JTAG peripheral supply if the card is not powered or plugged in. Otherwise if powered and plugged in, the 3v3 supply from the PCIe bus is used."
- note added: "PCIe 12v to 5v Supply"
- note removed: "Notes: ------------ This should allow the board to be powered from the jtag supply, and provide some reverse polarity protection. TODO: Size some mosfets, maybe dual package so8?"
- moved on the sheet: C100, C90, C91, C92, C93, C94, C95, C96, C97, C98, C99, L1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

Commit message: Third pass
Parts:
- added D6: POWER, LED_SMD:LED_0603_1608Metric, symbol Device:LED_Small
- added R71: 1k, Resistor_SMD:R_0402_1005Metric, symbol Device:R_Small
Connections:
- net +5V: now also R71.1
- net GND: now also D6.1 (K)
- new net: D6.2 (A), R71.2
Other:
- note added: "Power LED"
- company: (none) -> github.com/eggsampler
Changed lines of the file:
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@@
     (date "2024-01-01")
     (rev "1")
+    (company "github.com/eggsampler")
   )
   (junction (at 162.56 119.38) (diameter 0) (color 0 0 0 0)
@@
     (stroke (width 0) (type default))
   )
+  (wire (pts (xy 247.65 135.89) (xy 247.65 139.7))
+    (stroke (width 0) (type default))
+  )
   (wire (pts (xy 254 44.45) (xy 254 45.72))
     (stroke (width 0) (type default))
@@
     (stroke (width 0) (type default))
   )
+  (wire (pts (xy 247.65 114.3) (xy 247.65 118.11))
+    (stroke (width 0) (type default))
+  )
   (wire (pts (xy 134.62 127) (xy 162.56 127))
     (stroke (width 0) (type default))
@@
   )
   (wire (pts (xy 50.8 123.19) (xy 50.8 127))
+    (stroke (width 0) (type default))
+  )
+  (wire (pts (xy 247.65 123.19) (xy 247.65 130.81))
     (stroke (width 0) (type default))
   )
@@
   )
   (text "JTAG 3v3 Power Enable" (at 12.7 95.25 0)
+    (effects (font (size 3 3) (thickness 0.6) bold) (justify left bottom))
+  )
+  (text "Power LED" (at 212.09 95.25 0)
     (effects (font (size 3 3) (thickness 0.6) bold) (justify left bottom))
   )
@@
     )
   )
+  (symbol (lib_id "power:+5V") (at 247.65 114.3 0) (unit 1)
+    (in_bom yes) (on_board yes) (dnp no) (fields_autoplaced)
+    (property "Reference" "#PWR0180" (at 247.65 118.11 0)
+      (effects (font (size 1.27 1.27)) hide)
+    )
+    (property "Value" "+5V" (at 247.65 109.22 0)
+      (effects (font (size 1.27 1.27)))
+    )
+    (property "Footprint" "" (at 247.65 114.3 0)
+      (effects (font (size 1.27 1.27)) hide)
+    )
+    (property "Datasheet" "" (at 247.65 114.3 0)
+      (effects (font (size 1.27 1.27)) hide)
+    )
+    (pin "1")
+    (instances
+      (project "PCIeDMA"
+        (path "/e81b7940-99a9-4b7f-b36e-83163c2a41ea/11b53c35-cc79-4ae5-8f22-77aa75b8682b"
+          (reference "#PWR0180") (unit 1)
+        )
+      )
+    )
+  )
   (symbol (lib_id "power:GND") (at 99.06 135.89 0) (unit 1)
     (in_bom yes) (on_board yes) (dnp no) (fields_autoplaced)
@@
     )
   )
+  (symbol (lib_id "Device:LED_Small") (at 247.65 133.35 90) (unit 1)
+    (in_bom yes) (on_board yes) (dnp no)
+    (property "Reference" "D6" (at 248.92 132.08 90)
+      (effects (font (size 1.27 1.27)) (justify right))
+    )
+    (property "Value" "POWER" (at 248.92 133.35 90)
+      (effects (font (size 1 1)) (justify right))
+    )
+    (property "Footprint" "LED_SMD:LED_0603_1608Metric" (at 247.65 133.35 90)
+      (effects (font (size 1.27 1.27)) hide)
+    )
+    (property "Datasheet" "~" (at 247.65 133.35 90)
+      (effects (font (size 1.27 1.27)) hide)
+    )
+    (property "Rating" "5mA 1.6V" (at 248.92 134.62 90)
+      (effects (font (size 1 1)) (justify right))
+    )
+    (property "Size" "0603" (at 248.92 135.89 90)
+      (effects (font (size 1 1)) (justify right))
+    )
+    (pin "1")
+    (pin "2")
+    (instances
+      (project "PCIeDMA"
+        (path "/e81b7940-99a9-4b7f-b36e-83163c2a41ea/11b53c35-cc79-4ae5-8f22-77aa75b8682b"
+          (reference "D6") (unit 1)
+        )
+      )
+    )
+  )
   (symbol (lib_id "Device:C_Small") (at 173.99 123.19 0) (unit 1)
     (in_bom yes) (on_board yes) (dnp no)
@@
         (path "/e81b7940-99a9-4b7f-b36e-83163c2a41ea/11b53c35-cc79-4ae5-8f22-77aa75b8682b"
           (reference "R51") (unit 1)
+        )
+      )
+    )
+  )
+  (symbol (lib_id "Device:R_Small") (at 247.65 120.65 0) (unit 1)
+    (in_bom yes) (on_board yes) (dnp no)
+    (property "Reference" "R71" (at 248.92 118.11 0)
+      (effects (font (size 1.27 1.27)) (justify left))
+    )
+    (property "Value" "1k" (at 248.92 119.38 0)
+      (effects (font (size 1 1)) (justify left))
+    )
+    (property "Footprint" "Resistor_SMD:R_0402_1005Metric" (at 247.65 120.65 0)
+      (effects (font (size 1.27 1.27)) hide)
+    )
+    (property "Datasheet" "~" (at 247.65 120.65 0)
+      (effects (font (size 1.27 1.27)) hide)
+    )
+    (property "Rating" "1/16W" (at 248.92 120.65 0)
+      (effects (font (size 1 1)) (justify left))
+    )
+    (property "Tolerance" "1%" (at 248.92 121.92 0)
+      (effects (font (size 1 1)) (justify left))
+    )
+    (property "Size" "0402" (at 248.92 123.19 0)
+      (effects (font (size 1 1)) (justify left))
+    )
+    (pin "1")
+    (pin "2")
+    (instances
+      (project "PCIeDMA"
+        (path "/e81b7940-99a9-4b7f-b36e-83163c2a41ea/11b53c35-cc79-4ae5-8f22-77aa75b8682b"
+          (reference "R71") (unit 1)
         )
       )
@@
         )
       )
+    )
+  )
+  (symbol (lib_id "power:GND") (at 247.65 139.7 0) (unit 1)
+    (in_bom yes) (on_board yes) (dnp no) (fields_autoplaced)
+    (property "Reference" "#PWR0181" (at 247.65 146.05 0)
+      (effects (font (size 1.27 1.27)) hide)
+    )
+    (property "Value" "GND" (at 247.65 144.78 0)
+      (effects (font (size 1.27 1.27)))
+    )
+    (property "Footprint" "" (at 247.65 139.7 0)
+      (effects (font (size 1.27 1.27)) hide)
+    )
+    (property "Datasheet" "" (at 247.65 139.7 0)
+      (effects (font (size 1.27 1.27)) hide)
+    )
+    (pin "1")
+    (instances
+      (project "PCIeDMA"
+        (path "/e81b7940-99a9-4b7f-b36e-83163c2a41ea/11b53c35-cc79-4ae5-8f22-77aa75b8682b"
+          (reference "#PWR0181") (unit 1)
+        )
+      )

Commit message: another quick pass
Parts:
- added TP11, TP8, TP9: TestPoint, TestPoint:TestPoint_Pad_D2.0mm, symbol Connector:TestPoint
Connections:
- net +12V: now also TP11.1
- net +5V: now also TP9.1
- net +5V_JTAG: now also TP8.1
