File: SS_Connector.kicad_sch (KiCad schematic)
At the start: 6 parts, among them J4 USB_C_Receptacle, U3 TPD4EUSB30, U4 TPD4EUSB30, U5 TPD4EUSB30

Commit message: Routing and layout, first pass
Connections:
- net DM renamed DN
- net RX1n renamed RX1-
- net RX1p renamed RX1+
- net RX2n renamed RX2-
- net RX2p renamed RX2+
- net TX1n renamed TX1-
- net TX1p renamed TX1+
- net TX2n renamed TX2-
- net TX2p renamed TX2+
Changed lines of the file:
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@@
     (effects (font (size 1.27 1.27)) (justify left bottom))
   )
-  (hierarchical_label "RX1p" (shape bidirectional) (at 266.7 93.98 0) (fields_autoplaced)
+  (hierarchical_label "RX1+" (shape bidirectional) (at 266.7 93.98 0) (fields_autoplaced)
     (effects (font (size 1.27 1.27)) (justify left))
   )
-  (hierarchical_label "TX1p" (shape bidirectional) (at 266.7 101.6 0) (fields_autoplaced)
+  (hierarchical_label "TX1+" (shape bidirectional) (at 266.7 101.6 0) (fields_autoplaced)
     (effects (font (size 1.27 1.27)) (justify left))
   )
-  (hierarchical_label "TX2p" (shape bidirectional) (at 266.7 116.84 0) (fields_autoplaced)
+  (hierarchical_label "TX2+" (shape bidirectional) (at 266.7 116.84 0) (fields_autoplaced)
     (effects (font (size 1.27 1.27)) (justify left))
   )
-  (hierarchical_label "TX1n" (shape bidirectional) (at 266.7 99.06 0) (fields_autoplaced)
+  (hierarchical_label "TX1-" (shape bidirectional) (at 266.7 99.06 0) (fields_autoplaced)
     (effects (font (size 1.27 1.27)) (justify left))
   )
-  (hierarchical_label "TX2n" (shape bidirectional) (at 266.7 114.3 0) (fields_autoplaced)
+  (hierarchical_label "TX2-" (shape bidirectional) (at 266.7 114.3 0) (fields_autoplaced)
     (effects (font (size 1.27 1.27)) (justify left))
   )
-  (hierarchical_label "RX1n" (shape bidirectional) (at 266.7 91.44 0) (fields_autoplaced)
+  (hierarchical_label "RX1-" (shape bidirectional) (at 266.7 91.44 0) (fields_autoplaced)
     (effects (font (size 1.27 1.27)) (justify left))
   )
-  (hierarchical_label "RX2p" (shape bidirectional) (at 266.7 109.22 0) (fields_autoplaced)
+  (hierarchical_label "RX2+" (shape bidirectional) (at 266.7 109.22 0) (fields_autoplaced)
     (effects (font (size 1.27 1.27)) (justify left))
   )
@@
     (effects (font (size 1.27 1.27)) (justify left))
   )
-  (hierarchical_label "RX2n" (shape bidirectional) (at 266.7 106.68 0) (fields_autoplaced)
+  (hierarchical_label "RX2-" (shape bidirectional) (at 266.7 106.68 0) (fields_autoplaced)
     (effects (font (size 1.27 1.27)) (justify left))
   )
-  (hierarchical_label "DM" (shape bidirectional) (at 266.7 78.74 0) (fields_autoplaced)
+  (hierarchical_label "DN" (shape bidirectional) (at 266.7 78.74 0) (fields_autoplaced)
     (effects (font (size 1.27 1.27)) (justify left))
   )

Commit message: Third pass
Other:
- company: (none) -> github.com/eggsampler
Changed lines of the file:
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@@
     (date "2024-01-01")
     (rev "1")
+    (company "github.com/eggsampler")
   )
   (junction (at 146.05 38.1) (diameter 0) (color 0 0 0 0)
