File: TypeCMux.kicad_sch (KiCad schematic)
At the start: 16 parts, among them Q1 Q_NMOS_DGS, U6 HD3SS3220

Commit message: Routing and layout, first pass
Parts:
- removed C38: 0.47u, Capacitor_SMD:C_0402_1005Metric, symbol Device:C_Small
- removed Q1: Q_NMOS_DGS, Package_TO_SOT_SMD:SOT-23, symbol Device:Q_NMOS_DGS
- removed R22, R23: 10k, Resistor_SMD:R_0402_1005Metric, symbol Device:R_Small
- renumbered C39 to C38
Connections:
- net GND: now also U6.29 (ENn_CC)
- net +VCCO renamed +3.3V
- net ENn: no longer names the net of R21.2, U6.12 (ENn_MUX)
- net ENn: no longer U6.29 (ENn_CC)
- net RX1n renamed RX1-
- net RX1p renamed RX1+
- net RX2n renamed RX2-
- net RX2p renamed RX2+
- net TOD_C_n renamed TOD_C_N
- net TOD_C_p renamed TOD_C_P
- net TX1_C_n renamed TX1_C_N
- net TX1_C_p renamed TX1_C_P
- net TX1n renamed TX1-
- net TX1p renamed TX1+
- net TX2_C_n renamed TX2_C_N
- net TX2_C_p renamed TX2_C_P
- net TX2n renamed TX2-
- net TX2p renamed TX2+

Commit message: Second pass
Parts:
- R19: footprint Resistor_SMD:R_1206_3216Metric -> Resistor_SMD:R_0805_2012Metric; Rating 0.1W -> >0.1W; Size 1206 -> 0805
Changed lines of the file:
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@@
   (title_block
     (title "PCIeDMA")
-    (date "2023-02-14")
+    (date "2024-01-01")
     (rev "1")
   )
@@
       (effects (font (size 1 1)) (justify left))
     )
-    (property "Footprint" "Resistor_SMD:R_1206_3216Metric" (at 101.6 50.8 0)
+    (property "Footprint" "Resistor_SMD:R_0805_2012Metric" (at 101.6 50.8 0)
       (effects (font (size 1.27 1.27)) hide)
     )
@@
       (effects (font (size 1.27 1.27)) hide)
     )
-    (property "Rating" "0.1W" (at 100.33 50.8 0)
+    (property "Rating" ">0.1W" (at 100.33 50.8 0)
       (effects (font (size 1 1)) (justify left))
     )
@@
       (effects (font (size 1 1)) (justify left))
     )
-    (property "Size" "1206" (at 100.33 53.34 0)
-      (effects (font (size 1 1)) (justify left))
-    )
+    (property "Size" "0805" (at 100.33 53.34 0)
+      (effects (font (size 1 1)) (justify left))
+    )

Commit message: Third pass
Other:
- company: (none) -> github.com/eggsampler
Changed lines of the file:
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@@
     (date "2024-01-01")
     (rev "1")
+    (company "github.com/eggsampler")
   )
   (bus_alias "I2C" (members "SDA" "SCL" "INT"))
