File: USB_Data.kicad_sch (KiCad schematic)
At the start: 0 parts

Commit message: Routing and layout, first pass
Other:
- sheet FT601 ports: added DN; removed DM
- sheet Type C Mux ports: added RX1+, RX1-, RX2+, RX2-, TX1+, TX1-, TX2+, TX2-; removed RX1n, RX1p, RX2n, RX2p, TX1n, TX1p, TX2n, TX2p
- sheet Type C SS Connector ports: added DN, RX1+, RX1-, RX2+, RX2-, TX1+, TX1-, TX2+, TX2-; removed DM, RX1n, RX1p, RX2n, RX2p, TX1n, TX1p, TX2n, TX2p
Changed lines of the file:
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@@
       (effects (font (size 1.27 1.27)) (justify left))
     )
-    (pin "DM" bidirectional (at 152.4 82.55 180)
+    (pin "DN" bidirectional (at 152.4 82.55 180)
       (effects (font (size 1.27 1.27)) (justify left))
     )
@@
       (effects (font (size 1.27 1.27)) (justify right))
     )
-    (pin "TX1p" bidirectional (at 101.6 101.6 180)
+    (pin "TX1+" bidirectional (at 101.6 101.6 180)
       (effects (font (size 1.27 1.27)) (justify left))
     )
-    (pin "RX1p" bidirectional (at 101.6 96.52 180)
+    (pin "RX1+" bidirectional (at 101.6 96.52 180)
       (effects (font (size 1.27 1.27)) (justify left))
     )
-    (pin "TX1n" bidirectional (at 101.6 99.06 180)
+    (pin "TX1-" bidirectional (at 101.6 99.06 180)
       (effects (font (size 1.27 1.27)) (justify left))
     )
-    (pin "RX2n" bidirectional (at 101.6 104.14 180)
+    (pin "RX2-" bidirectional (at 101.6 104.14 180)
       (effects (font (size 1.27 1.27)) (justify left))
     )
-    (pin "TX2n" bidirectional (at 101.6 109.22 180)
+    (pin "TX2-" bidirectional (at 101.6 109.22 180)
       (effects (font (size 1.27 1.27)) (justify left))
     )
-    (pin "RX2p" bidirectional (at 101.6 106.68 180)
+    (pin "RX2+" bidirectional (at 101.6 106.68 180)
       (effects (font (size 1.27 1.27)) (justify left))
     )
-    (pin "RX1n" bidirectional (at 101.6 93.98 180)
+    (pin "RX1-" bidirectional (at 101.6 93.98 180)
       (effects (font (size 1.27 1.27)) (justify left))
     )
-    (pin "TX2p" bidirectional (at 101.6 111.76 180)
+    (pin "TX2+" bidirectional (at 101.6 111.76 180)
       (effects (font (size 1.27 1.27)) (justify left))
     )
@@
       (effects (font (size 1.27 1.27)) (justify right))
     )
-    (pin "DM" bidirectional (at 76.2 82.55 0)
+    (pin "DN" bidirectional (at 76.2 82.55 0)
       (effects (font (size 1.27 1.27)) (justify right))
     )
-    (pin "TX2n" bidirectional (at 76.2 109.22 0)
+    (pin "TX2-" bidirectional (at 76.2 109.22 0)
       (effects (font (size 1.27 1.27)) (justify right))
     )
-    (pin "RX1n" bidirectional (at 76.2 93.98 0)
+    (pin "RX1-" bidirectional (at 76.2 93.98 0)
       (effects (font (size 1.27 1.27)) (justify right))
     )
-    (pin "RX2n" bidirectional (at 76.2 104.14 0)
+    (pin "RX2-" bidirectional (at 76.2 104.14 0)
       (effects (font (size 1.27 1.27)) (justify right))
     )
-    (pin "RX2p" bidirectional (at 76.2 106.68 0)
+    (pin "RX2+" bidirectional (at 76.2 106.68 0)
       (effects (font (size 1.27 1.27)) (justify right))
     )
-    (pin "TX2p" bidirectional (at 76.2 111.76 0)
+    (pin "TX2+" bidirectional (at 76.2 111.76 0)
       (effects (font (size 1.27 1.27)) (justify right))
     )
-    (pin "RX1p" bidirectional (at 76.2 96.52 0)
+    (pin "RX1+" bidirectional (at 76.2 96.52 0)
       (effects (font (size 1.27 1.27)) (justify right))
     )
-    (pin "TX1n" bidirectional (at 76.2 99.06 0)
+    (pin "TX1-" bidirectional (at 76.2 99.06 0)
       (effects (font (size 1.27 1.27)) (justify right))
     )
-    (pin "TX1p" bidirectional (at 76.2 101.6 0)
+    (pin "TX1+" bidirectional (at 76.2 101.6 0)
       (effects (font (size 1.27 1.27)) (justify right))
     )

Commit message: Third pass
Other:
- company: (none) -> github.com/eggsampler
Changed lines of the file:
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@@
     (date "2024-01-01")
     (rev "1")
+    (company "github.com/eggsampler")
   )
   (wire (pts (xy 138.43 66.04) (xy 90.17 66.04))
