File: USB_JTAG.kicad_sch (KiCad schematic)
At the start: 26 parts, among them J2 USB_C_Receptacle_USB2.0, J3 Conn_01x09, U1 TPD4EUSB30, U2 CH347T, Y1 8MHz

Commit message: Routing and layout, first pass
Parts:
- removed J3: Conn_01x09, Connector_PinHeader_1.27mm:PinHeader_1x09_P1.27mm_Vertical, symbol Connector_Generic:Conn_01x09
- added J3: Conn_01x10, Connector_PinHeader_1.27mm:PinHeader_1x10_P1.27mm_Vertical, symbol Connector_Generic:Conn_01x10
Connections:
- net +3.3V: now also J3.9 (Pin_9)
- net +5V: now also J3.10 (Pin_10)
- net +5V_JTAG: now also J3.2 (Pin_2)
- net GND: now also J3.1 (Pin_1)
- net RST: now also J3.3 (Pin_3)
- net TCK_CONN: now also J3.5 (Pin_5)
- net TDI_CONN: now also J3.7 (Pin_7)
- net TDO_CONN: now also J3.6 (Pin_6)
- net TMS_CONN: now also J3.4 (Pin_4)
- net TRST_CONN: now also J3.8 (Pin_8)
Other:
- moved on the sheet: R10, R11, R14, R15

Commit message: Second pass
Other:
- note added: "JTAG"
- moved on the sheet: C25, C26, C27, C28, C29, D1, FB1, J2, J3, R10, R11, R12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

Commit message: Third pass
Connections:
- net TX: now reaches U2.3 (TXD1)
- net RX: now reaches U2.4 (RXD1)
- no-connect marks 7 -> 5
Other:
- company: (none) -> github.com/eggsampler
Changed lines of the file:
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@@
     (date "2024-01-01")
     (rev "1")
-  )
+    (company "github.com/eggsampler")
+  )
+  (bus_alias "SERIAL" (members "RX" "TX"))
   (junction (at 33.02 127) (diameter 0) (color 0 0 0 0)
   )
@@
   (no_connect (at 212.09 129.54))
   (no_connect (at 212.09 127))
-  (no_connect (at 212.09 111.76))
   (no_connect (at 48.26 119.38))
   (no_connect (at 48.26 116.84))
-  (no_connect (at 212.09 109.22))
   (bus_entry (at 270.51 93.98) (size 2.54 -2.54)
     (stroke (width 0) (type default))
@@
     (stroke (width 0) (type default))
   )
+  (bus_entry (at 273.05 106.68) (size -2.54 2.54)
+    (stroke (width 0) (type default))
+  )
+  (bus_entry (at 273.05 109.22) (size -2.54 2.54)
+    (stroke (width 0) (type default))
+  )
   (wire (pts (xy 25.4 127) (xy 33.02 127))
     (stroke (width 0) (type default))
@@
     (stroke (width 0) (type default))
   )
+  (wire (pts (xy 212.09 109.22) (xy 270.51 109.22))
+    (stroke (width 0) (type default))
+  )
   (bus (pts (xy 273.05 76.2) (xy 273.05 88.9))
     (stroke (width 0) (type default))
   )
+  (bus (pts (xy 273.05 106.68) (xy 273.05 109.22))
+    (stroke (width 0) (type default))
+  )
   (wire (pts (xy 113.03 71.12) (xy 113.03 76.2))
     (stroke (width 0) (type default))
@@
     (stroke (width 0) (type default))
   )
+  (bus (pts (xy 273.05 104.14) (xy 273.05 106.68))
+    (stroke (width 0) (type default))
+  )
   (wire (pts (xy 234.95 66.04) (xy 234.95 91.44))
     (stroke (width 0) (type default))
@@
     (stroke (width 0) (type default))
   )
-  (bus (pts (xy 274.32 76.2) (xy 273.05 76.2))
-    (stroke (width 0) (type default))
-  )
   (wire (pts (xy 48.26 101.6) (xy 48.26 104.14))
     (stroke (width 0) (type default))
@@
   )
   (wire (pts (xy 212.09 91.44) (xy 234.95 91.44))
+    (stroke (width 0) (type default))
+  )
+  (wire (pts (xy 270.51 111.76) (xy 212.09 111.76))
     (stroke (width 0) (type default))
   )
@@
     (effects (font (size 1.27 1.27)) (justify left bottom))
   )
+  (label "TX" (at 270.51 109.22 180) (fields_autoplaced)
+    (effects (font (size 1.27 1.27)) (justify right bottom))
+  )
   (label "RST" (at 223.52 31.75 180) (fields_autoplaced)
     (effects (font (size 1.27 1.27)) (justify right bottom))
@@
     (effects (font (size 1.27 1.27)) (justify left bottom))
   )
+  (label "RX" (at 270.51 111.76 180) (fields_autoplaced)
+    (effects (font (size 1.27 1.27)) (justify right bottom))
+  )
   (label "TDO_CONN" (at 219.71 39.37 180) (fields_autoplaced)
     (effects (font (size 1.27 1.27)) (justify right bottom))
@@
     (effects (font (size 1.27 1.27)) (justify left bottom))
   )
-  (hierarchical_label "{JTAG}" (shape bidirectional) (at 274.32 76.2 0) (fields_autoplaced)
+  (hierarchical_label "{SERIAL}" (shape bidirectional) (at 273.05 104.14 0) (fields_autoplaced)
     (effects (font (size 1.27 1.27)) (justify left))
   )
+  (hierarchical_label "{JTAG}" (shape bidirectional) (at 273.05 76.2 0) (fields_autoplaced)
+    (effects (font (size 1.27 1.27)) (justify left))
+  )
