File: User_IO.kicad_sch (KiCad schematic)
At the start: 8 parts, among them SW1 USER1, SW2 USER2

Commit message: Routing and layout, first pass
Parts:
- renumbered R26 to R24, R27 to R25, R28 to R26, R29 to R27

Commit message: Second pass
Parts:
- renumbered D3 to D2, D2 to D3
Changed lines of the file:
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@@
   (title_block
     (title "PCIeDMA")
-    (date "2023-02-14")
+    (date "2024-01-01")
     (rev "1")
   )
@@
   (symbol (lib_id "Device:LED_Small") (at 127 93.98 90) (unit 1)
     (in_bom yes) (on_board yes) (dnp no)
-    (property "Reference" "D2" (at 128.27 92.71 90)
+    (property "Reference" "D3" (at 128.27 92.71 90)
       (effects (font (size 1.27 1.27)) (justify right))
     )
@@
       (project "PCIeDMA"
         (path "/e81b7940-99a9-4b7f-b36e-83163c2a41ea/21232c02-71cb-435e-97ae-df589121e8b4"
-          (reference "D2") (unit 1)
+          (reference "D3") (unit 1)
         )
       )
@@
   (symbol (lib_id "Device:LED_Small") (at 152.4 93.98 90) (unit 1)
     (in_bom yes) (on_board yes) (dnp no)
-    (property "Reference" "D3" (at 153.67 92.71 90)
+    (property "Reference" "D2" (at 153.67 92.71 90)
       (effects (font (size 1.27 1.27)) (justify right))
     )
@@
       (project "PCIeDMA"
         (path "/e81b7940-99a9-4b7f-b36e-83163c2a41ea/21232c02-71cb-435e-97ae-df589121e8b4"
-          (reference "D3") (unit 1)
+          (reference "D2") (unit 1)
         )
       )

Commit message: Third pass
Other:
- company: (none) -> github.com/eggsampler
Changed lines of the file:
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@@
     (date "2024-01-01")
     (rev "1")
+    (company "github.com/eggsampler")
   )
   (junction (at 76.2 87.63) (diameter 0) (color 0 0 0 0)
